File: rainboard_neofighter/rainboard_newfighter.sch (KiCad schematic (older format))
At the start: 95 parts, among them J1 Conn_01x02, J10 Conn_01x03, J11 SDS-50J, J12 SDS-50J, J13 Conn_01x02, J14 Conn_01x02, J15 Conn_01x02, J16 Conn_01x02, J17 Conn_01x02, J18 Conn_01x02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

Commit message: send MINI IN opto signal through schmitt trigger
Connections:
- net Earth: now also J12.1, J12.3, U2.11 (5A), U2.13 (6A), XA1.GND6 (GND); no longer XA1.GND3 (GND)
- net GNDA: now also XA1.GND3 (GND); no longer XA1.GND6 (GND)
- net MIDI-IN: now also U2.8 (4Y); no longer R8.1, U3.4
- net at U2.5 (3A): now also R8.1, U3.4
- net at U2.6 (3Y): now also U2.9 (4A)
Other:
- moved on the sheet: C3
Changed lines of the file:
@@
 softpot-2
-$Comp
-L Arduino_Shields:Arduino_Mega2560_Shield XA1
-U 1 1 5F5FAE00
-P 2950 3200
-F 0 "XA1" H 2950 819 60  0000 C CNN
-F 1 "Arduino_Mega2560_Shield" H 2950 713 60  0000 C CNN
-F 2 "arduno_mega:Arduino_Mega2560_Shield" H 2950 607 60  0001 C CNN
-F 3 "https://store.arduino.cc/arduino-mega-2560-rev3" H 3650 5950 60  0001 C CNN
-	1    2950 3200
-	1    0    0    -1
-$EndComp
 $Comp
 L power:Earth #PWR0102
@@
 L Device:C C3
 U 1 1 603471DA
-P 20600 12800
-F 0 "C3" H 20715 12846 50  0000 L CNN
-F 1 "100nf" H 20715 12755 50  0000 L CNN
-F 2 "Capacitor_SMD:C_0603_1608Metric" H 20638 12650 50  0001 C CNN
-F 3 "~" H 20600 12800 50  0001 C CNN
-F 4 "C14663" H 20600 12800 50  0001 C CNN "LCSC"
-	1    20600 12800
-	1    0    0    -1
-$EndComp
-Connection ~ 20600 12950
-Wire Wire Line
-	20600 12950 20600 12850
-Wire Wire Line
-	20600 12450 20600 12650
-Text GLabel 20600 12450 0    50   Input ~ 0
+P 21150 13000
+F 0 "C3" H 21265 13046 50  0000 L CNN
+F 1 "100nf" H 21265 12955 50  0000 L CNN
+F 2 "Capacitor_SMD:C_0603_1608Metric" H 21188 12850 50  0001 C CNN
+F 3 "~" H 21150 13000 50  0001 C CNN
+F 4 "C14663" H 21150 13000 50  0001 C CNN "LCSC"
+	1    21150 13000
+	1    0    0    -1
+$EndComp
+Connection ~ 21150 13150
+Wire Wire Line
+	21150 13150 21150 13050
+Wire Wire Line
+	21150 12650 21150 12850
+Text GLabel 21150 12650 0    50   Input ~ 0
 5V
 $Comp
 L power:Earth #PWR0107
 U 1 1 603471D1
-P 20600 12950
-F 0 "#PWR0107" H 20600 12700 50  0001 C CNN
-F 1 "Earth" H 20600 12800 50  0001 C CNN
-F 2 "" H 20600 12950 50  0001 C CNN
-F 3 "~" H 20600 12950 50  0001 C CNN
-	1    20600 12950
+P 21150 13150
+F 0 "#PWR0107" H 21150 12900 50  0001 C CNN
+F 1 "Earth" H 21150 13000 50  0001 C CNN
+F 2 "" H 21150 13150 50  0001 C CNN
+F 3 "~" H 21150 13150 50  0001 C CNN
+	1    21150 13150
 	1    0    0    -1
 $EndComp
@@
 	1    0    0    -1
 $EndComp
-Text GLabel 15900 11800 2    50   Input ~ 0
+Text GLabel 20050 12550 2    50   Input ~ 0
 MIDI-IN
 Wire Wire Line
@@
 Wire Wire Line
 	15750 11900 15550 11900
-Wire Wire Line
-	15900 11800 15750 11800
 Connection ~ 15750 11800
 Wire Wire Line
@@
 Wire Wire Line
 	1650 5150 1650 5050
-Wire Wire Line
-	1150 4450 1650 4450
 $Comp
 L power:GNDA #PWR0104
@@
 	1    0    0    -1
 $EndComp
-Wire Wire Line
-	1350 4700 1500 4700
-Wire Wire Line
-	1500 4700 1500 4850
-Wire Wire Line
-	1500 4850 1650 4850
-Wire Wire Line
-	1650 4450 1650 4550
-Connection ~ 1650 4450
-Connection ~ 1650 4550
-Wire Wire Line
-	1650 4550 1650 4650
-Connection ~ 1650 4650
-Wire Wire Line
-	1650 4650 1650 4750
+$Comp
+L Arduino_Shields:Arduino_Mega2560_Shield XA1
+U 1 1 5F5FAE00
+P 2950 3200
+F 0 "XA1" H 2950 819 60  0000 C CNN
+F 1 "Arduino_Mega2560_Shield" H 2950 713 60  0000 C CNN
+F 2 "arduno_mega:Arduino_Mega2560_Shield" H 2950 607 60  0001 C CNN
+F 3 "https://store.arduino.cc/arduino-mega-2560-rev3" H 3650 5950 60  0001 C CNN
+	1    2950 3200
+	1    0    0    -1
+$EndComp
+Wire Wire Line
+	1350 4700 1350 4650
+Wire Wire Line
+	1350 4650 1650 4650
+Wire Wire Line
+	1550 4450 1550 4550
+Wire Wire Line
+	1550 4550 1650 4550
+Wire Wire Line
+	1150 4450 1550 4450
+Wire Wire Line
+	1550 4450 1650 4450
+Connection ~ 1550 4450
+Wire Wire Line
+	1550 4550 1550 4750
+Wire Wire Line
+	1550 4750 1650 4750
+Connection ~ 1550 4550
+Wire Wire Line
+	1550 4750 1550 4850
+Wire Wire Line
+	1550 4850 1650 4850
+Connection ~ 1550 4750
+Wire Wire Line
+	17400 11800 17400 12650
+Wire Wire Line
+	17400 12650 18550 12650
+Wire Wire Line
+	15750 11800 17400 11800
+Wire Wire Line
+	19950 12550 20050 12550
+Wire Wire Line
+	19950 12450 20500 12450
+Wire Wire Line
+	20500 12450 20500 13650
+Wire Wire Line
+	20500 13650 18050 13650
+Wire Wire Line
+	18050 13650 18050 12750
+Wire Wire Line
+	18050 12750 18550 12750
+Wire Wire Line
+	18550 13150 18550 12950
+Connection ~ 18550 13150
+Connection ~ 18550 12950
+Wire Wire Line
+	18550 12950 18550 12850
+Wire Wire Line
+	20800 11750 20800 11650
+Connection ~ 20800 11650
+Wire Wire Line
+	20800 11650 20800 11550
 $EndSCHEMATC
