File: rainboard_neofighter/rainboard_newfighter.kicad_pcb (KiCad board)
At the start: 2 copper layers, 260 x 253.6 mm, 98 parts, among them J1 Conn_01x02, J10 Conn_01x03, J11 SDS-50J, J12 SDS-50J, J13 Conn_01x02, J14 Conn_01x02, J15 Conn_01x02, J16 Conn_01x02, J17 Conn_01x02, J18 Conn_01x02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

Commit message: PCB v0.3
Connections:
- J12 pad 1: Earth -> Net-(J12-Pad1)
- J12 pad 3: Earth -> Net-(J12-Pad3)
Routing:
- net Earth: track 0.00 -> 1927.5 mm, vias 41 -> 0
- net Net-(J18-Pad2): track 185.0 -> 242.0 mm, vias 3 -> 2
- net Net-(J14-Pad2): track 200.2 -> 247.2 mm
- net Net-(J7-Pad2): track 205.1 -> 244.9 mm, vias 1 -> 3
- net softpot-1: track 47.5 -> 11.1 mm
- net Net-(J15-Pad2): track 206.9 -> 238.8 mm
- net Net-(J13-Pad2): track 212.3 -> 244.1 mm, vias 1 -> 2
- net button-35: track 247.2 -> 216.7 mm, vias 1 -> 2
- net BREF: track 67.6 -> 94.3 mm
- net button-12: track 128.4 -> 148.4 mm
- net button-06: track 144.7 -> 164.1 mm, vias 0 -> 1
- net 5V: track 223.3 -> 241.7 mm, vias 0 -> 1
- net button-01: track 156.7 -> 170.3 mm
- net button-13: track 110.3 -> 122.9 mm, vias 0 -> 1
- net button-36: track 115.3 -> 103.6 mm
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- removed copper zone on B.Cu, net Earth
- removed copper zone on F.Cu, net Earth
Other:
- board text added: "Rainboard V0.3"
- board text removed: "Rainboard V0.2"

Commit message: V0.3 candidate
Routing:
- net Earth: track 1927.5 -> 1868.6 mm, vias 0 -> 1
- net Net-(J18-Pad2): track 242.0 -> 196.9 mm
- net Net-(J14-Pad2): track 247.2 -> 207.0 mm, vias 2 -> 0
- net Net-(J7-Pad2): track 244.9 -> 211.0 mm, vias 3 -> 0
- net Net-(J13-Pad2): track 244.1 -> 212.1 mm
- net button-06: track 164.1 -> 143.4 mm, vias 1 -> 0
- net button-12: track 148.4 -> 132.0 mm, vias 1 -> 0
- net Net-(J15-Pad2): track 238.8 -> 224.2 mm, vias 2 -> 1
- net button-01: track 170.3 -> 156.6 mm, vias 1 -> 0
- net softpot-2: track 52.8 -> 39.8 mm
- net button-13: track 122.9 -> 110.3 mm, vias 1 -> 0
- net button-27: track 121.2 -> 132.3 mm, vias 1 -> 0
- net Net-(J16-Pad2): track 204.7 -> 193.6 mm
- net button-07: track 141.8 -> 130.9 mm, vias 2 -> 0
- net Net-(J1-Pad2): track 129.7 -> 120.7 mm, vias 1 -> 0
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