File: rainboard-pcb/rainboard_newfighter.kicad_pcb (KiCad board)
At the start: 2 copper layers, 260 x 253.6 mm, 98 parts, among them J1 Conn_01x02, J10 Conn_01x03, J11 SDS-50J, J12 SDS-50J, J13 Conn_01x02, J14 Conn_01x02, J15 Conn_01x02, J16 Conn_01x02, J17 Conn_01x02, J18 Conn_01x02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

Commit message: V0.4 exploratory work
Routing:
- net Earth: track 1868.6 -> 1895.0 mm

Commit message: start on v0.4 of PCB
Connections:
- J11 pad 1: Net-(J11-Pad1) -> (no net)
- J11 pad 2: Net-(J11-Pad2) -> (no net)
- J11 pad 3: Net-(J11-Pad3) -> (no net)
- J12 pad 1: Net-(J12-Pad1) -> (no net)
- J12 pad 3: Net-(J12-Pad3) -> (no net)
- U1 pad 19: Net-(U1-Pad19) -> (no net)
- U1 pad 20: Net-(U1-Pad20) -> (no net)
- U2 pad 10: Net-(U2-Pad10) -> (no net)
- U2 pad 12: Net-(U2-Pad12) -> (no net)
- XA1 pad 5V2: Net-(XA1-Pad5V2) -> (no net)
- XA1 pad A9: softpot-2 -> softpot-1
- XA1 pad D0: Net-(XA1-PadD0) -> (no net)
- XA1 pad D1: Net-(XA1-PadD1) -> (no net)
- XA1 pad D50: Net-(XA1-PadD50) -> (no net)
- XA1 pad D51: Net-(XA1-PadD51) -> (no net)
- XA1 pad D52: Net-(XA1-PadD52) -> (no net)
- XA1 pad D53: Net-(XA1-PadD53) -> (no net)
- XA1 pad GND4: Net-(XA1-PadGND4) -> (no net)
- XA1 pad IORF: Net-(XA1-PadIORF) -> (no net)
- XA1 pad MISO: Net-(XA1-PadMISO) -> (no net)
- XA1 pad MOSI: Net-(XA1-PadMOSI) -> (no net)
- XA1 pad RST1: Net-(XA1-PadRST1) -> (no net)
- XA1 pad RST2: Net-(XA1-PadRST2) -> (no net)
- XA1 pad SCK: Net-(XA1-PadSCK) -> (no net)
- XA1 pad VIN: Net-(XA1-PadVIN) -> (no net)
Routing:
- net softpot-1: track 6.88 -> 42.9 mm, vias 0 -> 2
- net softpot-2: track 39.8 -> 42.6 mm

Commit message: fix issues with buttons 25 and 28. Improved ground and power network
Parts:
- removed J17, J18: Conn_01x02, Connector_JST:JST_XH_B2B-XH-AM_1x02_P2.50mm_Vertical
Connections:
- J11 pad 1: (no net) -> Net-(J11-Pad1)
- J11 pad 2: (no net) -> Net-(J11-Pad2)
- J11 pad 3: (no net) -> Net-(J11-Pad3)
- J12 pad 1: (no net) -> Net-(J12-Pad1)
- J12 pad 3: (no net) -> Net-(J12-Pad3)
- U1 pad 19: (no net) -> Net-(U1-Pad19)
- U1 pad 20: (no net) -> Net-(U1-Pad20)
- U1 pad 27: Net-(J17-Pad2) -> button-28
- U1 pad 28: Net-(J18-Pad2) -> button-25
- U2 pad 10: (no net) -> Net-(U2-Pad10)
- U2 pad 12: (no net) -> Net-(U2-Pad12)
- XA1 pad 5V2: (no net) -> Net-(XA1-Pad5V2)
- XA1 pad D0: (no net) -> Net-(XA1-PadD0)
- XA1 pad D1: (no net) -> Net-(XA1-PadD1)
- XA1 pad D20: button-25 -> Net-(XA1-PadD20)
- XA1 pad D21: button-28 -> Net-(XA1-PadD21)
- XA1 pad D50: (no net) -> Net-(XA1-PadD50)
- XA1 pad D51: (no net) -> Net-(XA1-PadD51)
- XA1 pad D52: (no net) -> Net-(XA1-PadD52)
- XA1 pad D53: (no net) -> Net-(XA1-PadD53)
- XA1 pad GND4: (no net) -> Net-(XA1-PadGND4)
- XA1 pad IORF: (no net) -> Net-(XA1-PadIORF)
- XA1 pad MISO: (no net) -> Net-(XA1-PadMISO)
- XA1 pad MOSI: (no net) -> Net-(XA1-PadMOSI)
- XA1 pad RST1: (no net) -> Net-(XA1-PadRST1)
- XA1 pad RST2: (no net) -> Net-(XA1-PadRST2)
- XA1 pad SCK: (no net) -> Net-(XA1-PadSCK)
- XA1 pad VIN: (no net) -> Net-(XA1-PadVIN)
Routing:
- net Net-(J8-Pad2): track 229.8 -> 0.00 mm, vias 2 -> 0
- net Net-(J15-Pad2): track 224.2 -> 0.00 mm, vias 1 -> 0
- net button-35: track 219.0 -> 0.00 mm, vias 1 -> 0
- net Net-(J13-Pad2): track 212.1 -> 0.00 mm, vias 2 -> 0
- net Net-(J7-Pad2): track 211.0 -> 0.00 mm
- net Net-(J14-Pad2): track 207.0 -> 0.00 mm
- net Net-(J6-Pad2): track 198.8 -> 0.00 mm
- net Net-(J18-Pad2): track 196.9 -> 0.00 mm, vias 2 -> 0
- net Net-(J5-Pad2): track 195.6 -> 0.00 mm
- net Net-(J16-Pad2): track 193.6 -> 0.00 mm, vias 2 -> 0
- net Net-(J4-Pad2): track 187.5 -> 0.00 mm
- net button-11: track 184.0 -> 0.00 mm, vias 1 -> 0
- net button-18: track 167.5 -> 0.00 mm, vias 1 -> 0
- net Net-(J17-Pad2): track 165.1 -> 0.00 mm
- net Net-(J3-Pad2): track 161.5 -> 0.00 mm
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Other:
- board text added: "Rainboard V0.4"
- board text removed: "Rainboard V0.3"

Commit message: Autorouted v0.4 with thicker power and earth traces
Parts:
- added R11: 220R, Resistor_SMD:R_0603_1608Metric, F.Cu at (-33.2, 121.7)
- D1: footprint Diode_SMD:D_SMA -> diode:SODFL2513X100N
- R8: value 10k -> 4.7k
- U3: value EL357N(A)(TA)-G -> 6N138SDM; footprint opto_coupler:SOP254P700X200-4N -> opto_coupler2:COUPL_6N138SDM
- moved J1 109.4 mm to (-61.5, 88.0), turned to 120 degrees
- moved J16 108.7 mm to (62.7, 86.1), turned to 240 degrees
- moved J13 107.7 mm to (106.8, 9.38), turned to 240 degrees
- moved J4 106.9 mm to (-106.2, 11.3), turned to 120 degrees
- moved J2 100.2 mm to (-76.4, 62.4), turned to 120 degrees
- moved J15 100.0 mm to (77.4, 60.5), turned to 240 degrees
- moved J14 99.7 mm to (92.1, 34.9), turned to 240 degrees
- moved J3 99.3 mm to (-91.3, 36.9), turned to 120 degrees
- moved R1 31.0 mm to (46.5, 40.6), turned to 0 degrees
- moved R3 30.6 mm to (51.0, 38.3), turned to 0 degrees
- moved Je 29.0 mm to (61.7, 35.5), turned to 180 degrees
- moved R2 23.3 mm to (51.4, 63.5), turned to 0 degrees
- moved J10 19.2 mm to (61.3, 65.8), turned to 180 degrees
- moved D1 17.2 mm to (-19.0, 121.8)
- moved R4 16.5 mm to (46.2, 59.5), turned to 0 degrees
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- renumbered J9 to Je
Connections:
- R8 pad 2: 5V -> Earth
- U2 pad 5: Net-(R8-Pad1) -> Net-(R11-Pad1)
- U3 pad 1: Net-(D1-Pad1) -> (no net)
- U3 pad 2: Net-(D1-Pad2) -> Net-(D1-Pad1)
- U3 pad 3: Earth -> Net-(D1-Pad2)
- U3 pad 4: Net-(R8-Pad1) -> (no net)
Routing:
- net Net-(J8-Pad2): track 0.00 -> 247.3 mm, vias 0 -> 2
- net Net-(J7-Pad2): track 0.00 -> 235.4 mm, vias 0 -> 1
- net button-25: track 0.00 -> 214.6 mm, vias 0 -> 2
- net Net-(J6-Pad2): track 0.00 -> 214.4 mm, vias 0 -> 2
- net button-35: track 0.00 -> 201.7 mm
- net Net-(J5-Pad2): track 0.00 -> 197.2 mm, vias 0 -> 1
- net button-11: track 0.00 -> 185.9 mm
- net button-18: track 0.00 -> 178.1 mm
- net Net-(J13-Pad2): track 0.00 -> 174.6 mm, vias 0 -> 2
- net Net-(J14-Pad2): track 0.00 -> 167.8 mm
- net button-01: track 0.00 -> 164.3 mm
- net button-05: track 0.00 -> 152.5 mm
- net button-02: track 0.00 -> 148.9 mm
- net button-03: track 0.00 -> 148.4 mm
- net button-04: track 0.00 -> 148.3 mm
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Other:
- board text added: "MIDI IN"
- board text added: "MIDI OUT"
