File: rainboard-pcb/kicad_proj/rainboard_newfighter/OFFBOARDBUTTONS.sch (KiCad schematic (older format))
At the start: 4 parts

Commit message: Schematic nearly finalized; PCB / footprint started
-Schematic is nearly finished. Needs some footprint associations and verifications.
-A few open questions remain.
-some lib updates to go w/ sch improvements
-
Parts:
- added C45, C47, C49, C50, C51, C52, C53, C54, C55, C56: 10uF 25V, Capacitor_SMD:C_1206_3216Metric, symbol lib_symbol:C
- added J10, J12, J14, J15, J16, J17, J18, J19, J20, J21: Conn_01x05_Male, symbol Connector:Conn_01x05_Male
- gave numbers to parts that had none: 4
Connections:
- net GND: now also J11.3 (Pin_3), J13.3 (Pin_3), C45.2, C47.2, C49.2, C50.2, C51.2, C52.2, C53.2, C54.2, C55.2, C56.2, J10.3 (Pin_3), J12.3 (Pin_3), J14.3 (Pin_3), J15.3 (Pin_3), J16.3 (Pin_3), J17.3 (Pin_3), J18.3 (Pin_3), J19.3 (Pin_3), J20.3 (Pin_3), J21.3 (Pin_3)
- net OFFBoardButton/DOUT: no longer J11.2 (Pin_2), J13.4 (Pin_4)
- net OFFBoardButton/GND: no longer J11.3 (Pin_3)
- net VLED: now also C45.1, C47.1, C49.1, C50.1, C51.1, C52.1, C53.1, C54.1, C55.1, C56.1, J10.5 (Pin_5), J12.5 (Pin_5), J14.5 (Pin_5), J15.5 (Pin_5), J16.5 (Pin_5), J17.5 (Pin_5), J18.5 (Pin_5), J19.5 (Pin_5), J20.5 (Pin_5), J21.5 (Pin_5)
- net sheet602A3A4D/DOUT: no longer J13.2 (Pin_2)
- net sheet602A3A4D/GND: no longer J13.3 (Pin_3)
- net BTN-X renamed BTNX-1
- net BTN-X+1 renamed BTNX-2
- new net: J15.2 (Pin_2), J17.4 (Pin_4)
- new net: J13.2 (Pin_2), J15.4 (Pin_4)
- new net: J17.2 (Pin_2), J19.4 (Pin_4)
- new net: J19.2 (Pin_2), J21.4 (Pin_4)
- new net: J10.4 (Pin_4), J21.2 (Pin_2)
- new net: J10.2 (Pin_2), J12.4 (Pin_4)
- new net: J12.2 (Pin_2), J14.4 (Pin_4)
- new net: J14.2 (Pin_2), J16.4 (Pin_4)
- new net: J16.2 (Pin_2), J18.4 (Pin_4)
- new net: J18.2 (Pin_2), J20.4 (Pin_4)
- new net: J11.2 (Pin_2), J13.4 (Pin_4)
- new net BTNX-10: J16.1 (Pin_1)
- new net BTNX-11: J18.1 (Pin_1)
- new net BTNX-12: J20.1 (Pin_1)
- new net BTNX-3: J15.1 (Pin_1)
- new net BTNX-4: J17.1 (Pin_1)
- new net BTNX-5: J19.1 (Pin_1)
- new net BTNX-6: J21.1 (Pin_1)
- new net BTNX-7: J10.1 (Pin_1)
- new net BTNX-8: J12.1 (Pin_1)
- new net BTNX-9: J14.1 (Pin_1)
- new net FINAL_DOUT: J20.2 (Pin_2)
Other:
- note added: "Place 10uF caps near each\npair of headers\n"
- note added: "TODO SELECT CONNECTOR\n"
- note removed: "Place caps near each\npair of headers\n"
- note removed: "TODO SELECT CONNECTOR\nTODO X12"
- moved on the sheet: C46, C48, J11, J13
