File: rainboard-pcb/kicad_proj/rainboard_newfighter/PCBMountButtons.sch (KiCad schematic (older format))
At the start: 26 parts

Commit message: Schematic nearly finalized; PCB / footprint started
-Schematic is nearly finished. Needs some footprint associations and verifications.
-A few open questions remain.
-some lib updates to go w/ sch improvements
-
Parts:
- added R100, R101, R102, R104, R105, R106, R107, R109, R110, R111, R112, R114, R115, R116, R117, R119, R120, R121, R123, R124, R125, R127, R128, R129, R74, R75, R76, R77, R79, R80, R81, R82, R84, R85, R86, R87, R89, R90, R91, R92, R94, R95, R96, R97, R99: 210R, Resistor_SMD:R_0805_2012Metric, symbol Device:R
- C88, C89, C90, C91: renamed from C?; footprint (none) -> Capacitor_SMD:CP_Elec_10x10
- gave numbers to parts that had none: 22
Connections:
- net FINAL_DOUT: now also R114.2
- net sheet61AD1E9C/DIN renamed sheet5FFC6464/DIN
- new net sheet5FFC6464/DOUT: R77.1
- new net sheet5FFC646C/DIN: R77.2
- new net sheet5FFC646C/DOUT: R82.1
- new net sheet5FFC6480/DIN: R82.2
- new net sheet5FFC6480/DOUT: R87.1
- new net sheet5FFC6494/DIN: R87.2
- new net sheet5FFC6494/DOUT: R92.1
- new net sheet5FFC64B5/DIN: R92.2
- new net sheet5FFC64B5/DOUT: R97.1
- new net sheet5FFC64BB/DIN: R97.2
- new net sheet5FFC64BB/DOUT: R102.1
- new net sheet5FFC64CF/DIN: R102.2
- new net sheet5FFC64CF/DOUT: R107.1
- new net sheet5FFC64F0/DIN: R107.2
- new net sheet5FFC64F0/DOUT: R112.1
- new net sheet5FFC64F7/DIN: R112.2
- new net sheet5FFC64F7/DOUT: R117.1
- new net sheet5FFC6517/DIN: R117.2
- new net sheet5FFC6517/DOUT: R121.1
- new net sheet5FFC651D/DIN: R121.2
- new net sheet5FFC651D/DOUT: R125.1
- new net sheet5FFC6531/DIN: R125.2
- new net sheet5FFC6531/DOUT: R129.1
- new net sheet5FFD985B/DIN: R129.2
- new net sheet5FFD985B/DOUT: R76.1
- new net sheet5FFD9863/DIN: R76.2
- new net sheet5FFD9863/DOUT: R81.1
- new net sheet5FFD9877/DIN: R81.2
- new net sheet5FFD9877/DOUT: R86.1
- new net sheet5FFD988B/DIN: R86.2
- new net sheet5FFD988B/DOUT: R91.1
- new net sheet5FFD98AC/DIN: R91.2
- new net sheet5FFD98AC/DOUT: R96.1
- new net sheet5FFD98B2/DIN: R96.2
- new net sheet5FFD98B2/DOUT: R101.1
- new net sheet5FFD98C6/DIN: R101.2
- new net sheet5FFD98C6/DOUT: R106.1
- new net sheet5FFD98E7/DIN: R106.2
- new net sheet5FFD98E7/DOUT: R111.1
- new net sheet5FFD98EE/DIN: R111.2
- new net sheet5FFD98EE/DOUT: R116.1
- new net sheet5FFD990E/DIN: R116.2
- new net sheet5FFD990E/DOUT: R120.1
- new net sheet5FFD9914/DIN: R120.2
- new net sheet5FFD9914/DOUT: R124.1
- new net sheet5FFD9928/DIN: R124.2
- new net sheet5FFD9928/DOUT: R128.1
- new net sheet5FFFA930/DIN: R128.2
- new net sheet5FFFA930/DOUT: R75.1
- new net sheet5FFFA938/DIN: R75.2
- new net sheet5FFFA938/DOUT: R80.1
- new net sheet5FFFA94C/DIN: R80.2
- new net sheet5FFFA94C/DOUT: R85.1
- new net sheet5FFFA960/DIN: R85.2
- new net sheet5FFFA960/DOUT: R90.1
- new net sheet5FFFA981/DIN: R90.2
- new net sheet5FFFA981/DOUT: R95.1
- new net sheet5FFFA987/DIN: R95.2
- new net sheet5FFFA987/DOUT: R100.1
- new net sheet5FFFA99B/DIN: R100.2
- new net sheet5FFFA99B/DOUT: R105.1
- new net sheet5FFFA9BC/DIN: R105.2
- new net sheet5FFFA9BC/DOUT: R110.1
- new net sheet5FFFA9C3/DIN: R110.2
- new net sheet5FFFA9C3/DOUT: R115.1
- new net sheet5FFFA9E3/DIN: R115.2
- new net sheet5FFFA9E3/DOUT: R119.1
- new net sheet5FFFA9E9/DIN: R119.2
- new net sheet5FFFA9E9/DOUT: R123.1
- new net sheet5FFFA9FD/DIN: R123.2
- new net sheet5FFFA9FD/DOUT: R127.1
- new net sheet6001C156/DIN: R127.2
- new net sheet6001C156/DOUT: R74.1
- new net sheet6001C15E/DIN: R74.2
- new net sheet6001C15E/DOUT: R79.1
- new net sheet6001C172/DIN: R79.2
- new net sheet6001C172/DOUT: R84.1
- new net sheet6001C186/DIN: R84.2
- new net sheet6001C186/DOUT: R89.1
- new net sheet6001C1A7/DIN: R89.2
- new net sheet6001C1A7/DOUT: R94.1
- new net sheet6001C1AD/DIN: R94.2
- new net sheet6001C1AD/DOUT: R99.1
- new net sheet6001C1C1/DIN: R99.2
- new net sheet6001C1C1/DOUT: R104.1
- new net sheet6001C1E2/DIN: R104.2
- new net sheet6001C1E2/DOUT: R109.1
- new net sheet6001C1E9/DIN: R109.2
- new net sheet6001C1E9/DOUT: R114.1
Other:
- note added: "#17"
- note added: "#29"
- note added: "#41"
- note added: "#5"
- note added: "#53"
- note added: "#61"
- note removed: "#1"
- note removed: "#13\n"
- note removed: "#8\n"
- note removed: "#9\n"
- note removed: "#\n"
- note removed: "TODO rename to button-n"
- note removed: "TODO, 61 OF EM"
- note removed: "TODO, more of these ???"
