File: rainboard-pcb/kicad_proj/rainboard_newfighter/PCBMountButtons.sch (KiCad schematic (older format))
At the start: 74 parts

Commit message: prelim place & route
deleted extra R's layout & sch
Parts:
- removed R100, R101, R102, R103, R104, R105, R106, R107, R108, R109, R110, R111, R112, R113, R54, R55, R56, R57, R58, R59, R60, R61, R62, R63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: 210R, Resistor_SMD:R_0805_2012Metric, symbol Device:R
