File: rainboard-pcb/kicad_proj/rainboard_newfighter/rainboard_newfighter.sch (KiCad schematic (older format))
At the start: 101 parts, among them J10 Conn_01x03, J9 Conn_01x03

Commit message: Starts new revision, fixes lib path
Input filtering/protection/etc. ; lots of schematic symbols, most of them paired to a footprint. All saved to project library.

A few button/RGB combos placed, didn't go 60x yet in case it needs a change.
Parts:
- added C? (x4): 100nf, Capacitor_SMD:C_0603_1608Metric, symbol Device:C
- added C? (x4): 1uF 25V, Capacitor_SMD:C_0805_2012Metric, symbol lib_symbol:C
- added C? (x4): 1uF 25V, symbol lib_symbol:C
- added C? (x3): 470uF 25V, symbol lib_symbol:CP
- added C? (x9): 10uF 25V, Capacitor_SMD:C_1206_3216Metric, symbol lib_symbol:C
- added D? (x6): WS2812B, LED_SMD:LED_WS2812B_PLCC4_5.0x5.0mm_P3.2mm, symbol lib_symbol:WS2812B
- added D? (x2): 12Vw, Diode_SMD:D_SMA, symbol lib_symbol:D_Zener
- added D?: 5Vw, Diode_SMD:D_SMA, symbol lib_symbol:D_Zener
- added D? (x3): 40V 1A, Diode_SMD:D_SOD-123, symbol lib_symbol:D_Schottky
- added F?: 20V 3A, Fuse:Fuse_1812_4532Metric, symbol lib_symbol:Polyfuse
- added F?: 15V .5A, Fuse:Fuse_1812_4532Metric, symbol lib_symbol:Polyfuse
- added FB? (x2): Ferrite_Bead, symbol lib_symbol:Ferrite_Bead
- added FB?: 3A Ferrite, symbol lib_symbol:Ferrite_Bead
- added J?: EJ508A, Connector_BarrelJack:BarrelJack_Horizontal, symbol lib_symbol:Barrel_Jack_Switch
- added J?: C46390, symbol lib_symbol:USB_B_Micro
- added L? (x2): L, symbol lib_symbol:L
- added L? (x2): 10uH .5Ohm, symbol lib_symbol:L
- added Q?: 30V 10mOhm, Package_SO:PowerPAK_SO-8_Single, symbol lib_symbol:NMOS_SGD_123_4_5
- added R? (x6): 220R, Resistor_SMD:R_0603_1608Metric, symbol lib_symbol:R
- added R? (x5): 100k, Resistor_SMD:R_0603_1608Metric, symbol Device:R
- added R?: 19.1k, Resistor_SMD:R_0603_1608Metric, symbol Device:R
- added R? (x2): 22R, Resistor_SMD:R_0603_1608Metric, symbol lib_symbol:R
- added SW? (x5): SANWA-OBSF24, symbol lib_symbol:SANWA-OBSF24
- added U?: RT8298, Package_SO:SOIC-8-1EP_3.9x4.9mm_P1.27mm_EP2.41x3.3mm_ThermalVias, symbol lib_symbol:RT8298
- added U?: ATmega16U2-MU, Package_DFN_QFN:QFN-32-1EP_5x5mm_P0.5mm_EP3.1x3.1mm, symbol MCU_Microchip_ATmega:ATmega16U2-MU
- added U?: ATmega2560-16AU, Package_QFP:TQFP-100_14x14mm_P0.5mm, symbol lib_symbol:ATmega2560-16AU
Connections:
- net labels added: 12V_FILT, 5V_MCU, 5V_POW, 5V_USB, BARREL_DETECT, BTN, BTN1, BTN2, BTN4, BTN5, D+, D-, GND, LED_CTRL, LED_CTRL_, LED_CTRL_1, LED_CTRL_2, LED_CTRL_3, LED_CTRL_4, LED_CTRL_5, LED_CTRL_6, VLED
- wire segments 159 -> 358
Other:
- note added: "12V - 5V; 5A Buck"
- note added: "50mA each LED, \nx60 = 3A minimum"
- note added: "ARDUINO BOOTLOADER"
- note added: "BARREL POWER \nDETECT"
- note added: "BUTTON"
- note added: "BUTTON 1"
- note added: "BUTTON 2"
- note added: "BUTTON 3"
- note added: "BUTTON 4"
- note added: "BUTTON 5"
- note added: "BUTTONS"
- note added: "Barrel Jack Input"
- note added: "Diode OR for MCU Power"
- note added: "Filter and Surge & Reverse Polarity Protection"
- note added: "MAIN MCU"
- note added: "Micro USB Input"
- note added: "Place if Ceramic Caps\nMake noise from RBG PWM"
- note added: "Schottky Optional for\nBetter Efficiency"
- note added: "TODO data protection"
- note added: "TODO double check footprint, \nusing kicad lib generic"
- note added: "TODO footprint"
- moved on the sheet: SW?

Commit message: Schematic improvements; LED/buttons and MCU
Creates subsheet for on-board LED/BUTTON and off-board LED/button
most electrical connections of 2560.
most electrical connections of arudino front end
most electrical connections of LED controller.
Adds ESD protection to MIDI

lots of TODO/questions in text to see what progress remains.
Parts:
- removed D1: D, diode:SODFL2513X100N, symbol Device:D
- removed D? (x6): WS2812B, LED_SMD:LED_WS2812B_PLCC4_5.0x5.0mm_P3.2mm, symbol lib_symbol:WS2812B
- removed R7, R? (x2): 220R, Resistor_SMD:R_0603_1608Metric, symbol Device:R
- removed R? (x6): 220R, Resistor_SMD:R_0603_1608Metric, symbol lib_symbol:R
- removed SW? (x6): SANWA-OBSF24, symbol lib_symbol:SANWA-OBSF24
- added C? (x5): 100nf, Capacitor_SMD:C_0603_1608Metric, symbol Device:C
- added C? (x3): 1uF 25V, Capacitor_SMD:C_0805_2012Metric, symbol lib_symbol:C
- added C?: 470uF 25V, symbol lib_symbol:CP
- added C? (x4): 22PF, Capacitor_SMD:C_0603_1608Metric, symbol Device:C
- added D? (x5): 5Vw, Package_TO_SOT_SMD:SOT-23, symbol lib_symbol:D_Zener_x2_ACom_KKA
- added J? (x3): PH2-06-UA, symbol lib_symbol:Conn_02x03_Odd_Even
- added L?: 10uH .5Ohm, symbol lib_symbol:L
- added R? (x3): 19.1k, Resistor_SMD:R_0603_1608Metric, symbol Device:R
- added R? (x7): 11R, Resistor_SMD:R_0603_1608Metric, symbol lib_symbol:R
- added R? (x4): 210R, Resistor_SMD:R_0805_2012Metric, symbol Device:R
- added R? (x2): DNP-210R, Resistor_SMD:R_0603_1608Metric, symbol Device:R
- added R?: 4.7k, Resistor_SMD:R_0603_1608Metric, symbol Device:R
- added U?: ATmega16U2-MU, Package_DFN_QFN:QFN-32-1EP_5x5mm_P0.5mm_EP3.1x3.1mm, symbol MCU_Microchip_ATmega:ATmega16U2-MU
- added Y? (x2): Crystal, Crystal:Crystal_HC49-U_Vertical, symbol Device:Crystal
- added Y?: 16MHz CSTNE16M0V530000R0, Crystal:Resonator_SMD_muRata_CSTxExxV-3Pin_3.0x1.1mm, symbol Device:Resonator
- R5: value 220R -> 210R; footprint Resistor_SMD:R_0603_1608Metric -> Resistor_SMD:R_0805_2012Metric; LCSC C22962 -> C228630
- R? (x2): value 22R -> 11R; LCSC C269708 -> C227565
Connections:
- net labels added: 5VA_MCU, M8RXD, M8TXD, MCU1-MCU3_TX, MCU1_LED_CTRL, MCU1_MISO, MCU1_RST, MCU1_SCK, MCU2_LED_CTRL, MCU2_MISO2, MCU2_MOSI2, MCU2_RST, MCU2_SCK2, MCU3_LED_CTRL, MCU3_MISO3, MCU3_MOSI3, MCU3_RST, MCU3_SCK3, MCU_MOSI, PROG_CTRL_1, PROG_CTRL_2, button-25, button-27, button-28, button-35, button-X-1, button-X-10, button-X-11, button-X-12, button-X-2, button-X-3, button-X-4, button-X-5, button-X-6, button-X-7, button-X-8, button-X-9
- net labels removed: BTN, BTN1, BTN2, BTN4, BTN5, LED_CTRL, LED_CTRL_, LED_CTRL_1, LED_CTRL_2, LED_CTRL_3, LED_CTRL_4, LED_CTRL_5, LED_CTRL_6
- wire segments 358 -> 525
Other:
- note added: "50mA each LED, \nx12 = 600mA minimum"
- note added: "50mA each LED, \nx61 = 3A minimum"
- note added: "ARDUINO INTERFACE MCU"
- note added: "ICSP"
- note added: "LED CONTROLLER MCU"
- note added: "OFF-BOARD BUTTONS\n"
- note added: "PCB MOUNT\nRGB BUTTONS"
- note added: "QUESTION, ASIDE FROM INPUT/OUTPUT CONNECTORS, WHAT ELSE NEEDS ESD PROTECTION?\nEVERY BUTTON/GPIO WOULD BE VERY MANY, MAYBE BEST TO JUST HAVE THE MCUs/ETC ON THE FAR SIDE SO USER CAN'T REACH MOST INPUTS"
- note added: "QUESTION, DO WE NEED RESET BUTTONS ON BOARD?\nTODO, ADD"
- note added: "QUESTION,\nADC OR GPIO FOR THIS?\nEITHER WORKS, \nADC WILL REQUIRE MOVING SOME BUTTONS"
- note added: "QUESTION,\nNEED BOARD LEVEL DISCRETE LEDS?"
- note added: "QUESTION,\nTIE SHIELD TO GND?\nTODO, FIGURE OUT"
- note added: "QUESTION:\nMICRO OK, OR MINI?"
- note added: "TODO"
- note added: "TODO FIND A XTAL/RESONATOR THAT CAN DO BOTH MCUS ??"
- note added: "TODO, HOOK THESE UP FOR PROGRAMMING CONTROL\nTODO, DESIGN FET/RELAY CIRCUIT\n(REPLACES JUMPERS)"
- note added: "TODO, IS DIODE TO 5V ON RESET NEEDED?!??"
- note added: "TODO, JUMPER JP5: PB4-7"
- note added: "TODO,\nCAN PROBABLY GET AWAY WITHOUT OSCILLATOR HERE,\nDOUBLE CHECK ACCURACY"
- note added: "TODO,\nRESET_EN JUMPER??"
- note added: "TODO\nFIGURE OUT IF UVCC IS CORRECTLY SETUP HERE"
- note added: "TODO\nUGND/PAD/GND GNDS AND JUMPERS ARE WEIRD ON MEGA??"
- note removed: "50mA each LED, \nx60 = 3A minimum"
- note removed: "ARDUINO BOOTLOADER"
- note removed: "BUTTON"
- note removed: "BUTTON 1"
- note removed: "BUTTON 2"
- note removed: "BUTTON 3"
- note removed: "BUTTON 4"
- note removed: "BUTTON 5"
- note removed: "BUTTONS"
- note removed: "TODO data protection"
- moved on the sheet: C2, C4, R1, R2, R4, R5, R?, SW?, U?, U?G

Commit message: Schematic nearly finalized; PCB / footprint started
-Schematic is nearly finished. Needs some footprint associations and verifications.
-A few open questions remain.
-some lib updates to go w/ sch improvements
-
Parts:
- removed FB?: Ferrite_Bead, symbol lib_symbol:Ferrite_Bead
- removed J10, J9: Conn_01x03, Connector_JST:JST_XH_B3B-XH-AM_1x03_P2.50mm_Vertical, symbol Connector_Generic:Conn_01x03
- removed J? (x2): SDS-50J, symbol Connector:Conn_01x06_Female
- removed L?: L, symbol lib_symbol:L
- removed R? (x2): DNP-210R, Resistor_SMD:R_0603_1608Metric, symbol Device:R
- removed SW? (x60): SANWA-OBSF24, symbol lib_symbol:SANWA-OBSF24
- removed SW? (x16): META-BUTTON, symbol lib_symbol:META-BUTTON
- added C28: 1uF 25V, Capacitor_SMD:C_0805_2012Metric, symbol lib_symbol:C
- added C29, C31, C40, C44: 100nf, Capacitor_SMD:C_0603_1608Metric, symbol Device:C
- added D14, D17, D18, D6: 40V 1A, Diode_SMD:D_SOD-123, symbol lib_symbol:D_Schottky
- added D7, D8: 5Vw, Package_TO_SOT_SMD:SOT-23, symbol lib_symbol:D_Zener_x2_ACom_KKA
- added D9: 5Vw, Diode_SMD:D_SMA, symbol lib_symbol:D_Zener
- added FB1: 4A Ferrite, Inductor_SMD:L_1206_3216Metric, symbol lib_symbol:Ferrite_Bead
- added J3, J4: Conn_01x03, Connector_JST:JST_XH_B3B-XH-AM_1x03_P2.50mm_Vertical, symbol lib_symbol:Conn_01x03
- added J6, J7: SDS-50J, SDS-50J:CUI_SDS-50J, symbol lib_symbol:SDS-50J
- added JP1, JP2, JP3, JP4, JP5: Jumper, Jumper:SolderJumper-2_P1.3mm_Bridged_Pad1.0x1.5mm, symbol lib_symbol:Jumper
- added L1: 27uH, Inductor_SMD:L_Bourns_SRR1210A, symbol lib_symbol:L
- added Q1, Q2: DUAL 30V NMOS, Package_TO_SOT_SMD:SOT-363_SC-70-6, symbol lib_symbol:Q_DUAL_NMOS_S1G1D2S2G2D1
- added R18: DNP-4.7k, Resistor_SMD:R_0603_1608Metric, symbol Device:R
- added R19, R32, R33, R41: 4.7k, Resistor_SMD:R_0603_1608Metric, symbol Device:R
- added R20, R22, R36, R37: 11R, Resistor_SMD:R_0603_1608Metric, symbol lib_symbol:R
- added R24, R40: 19.1k, Resistor_SMD:R_0603_1608Metric, symbol Device:R
- added R26: DNP-210R, Resistor_SMD:R_0805_2012Metric, symbol Device:R
- added TP1, TP10, TP11, TP12, TP13, TP14, TP15, TP16, TP17, TP18, TP19, TP2, TP20, TP21, TP22, TP23, TP24, TP25, TP26, TP3, TP4, TP5, TP6, TP7, TP8, TP9: TestPoint, TestPoint:TestPoint_Pad_1.0x1.0mm, symbol lib_symbol:TestPoint
- C11, C13, C23, C5: renamed from C?; footprint (none) -> Capacitor_SMD:C_0805_2012Metric
- C14, C20, C32, C38: renamed from C?; footprint (none) -> Capacitor_SMD:CP_Elec_10x10
- FB2: renamed from FB?; value 3A Ferrite -> 4A Ferrite; footprint (none) -> Inductor_SMD:L_1206_3216Metric
- FB3: renamed from FB?; value Ferrite_Bead -> 4A Ferrite; footprint (none) -> Inductor_SMD:L_1206_3216Metric; PN MH2029-300Y -> MFBW1V3216-090-R
- L3: renamed from L?; value L -> 27uH; footprint (none) -> Inductor_SMD:L_Bourns_SRR1210A; PN (none) -> SRR1210-270M
- U4: renamed from U?; footprint (none) -> Package_SO:TSSOP-14_4.4x5mm_P0.65mm; PN (none) -> 74HC14PW-Q100,118
- gave numbers to parts that had none: 83
Connections:
- net labels added: BTN10, BTN11, BTN12, BTN13, BTN14, BTN15, BTN16, BTN17, BTN18, BTN19, BTN1a, BTN1b, BTN20, BTN21, BTN22, BTN23, BTN24, BTN25, BTN26, BTN27, BTN28, BTN29, BTN2a, BTN2b, BTN30, BTN31, BTN32, BTN33, BTN34, BTN35, BTN36, BTN37, BTN38, BTN39, BTN3a, BTN3b, BTN40, BTN41, BTN42, BTN43, BTN44, BTN45, BTN46, BTN47, BTN48, BTN49, BTN4a, BTN4b, BTN5, BTN50, BTN51, BTN52, BTN53, BTN54, BTN55, BTN56, BTN57, BTN58, BTN59, BTN6, BTN60, BTN61, BTN7, BTN8, BTN9, BTNX-1, BTNX-10, BTNX-11, BTNX-12, BTNX-2, BTNX-3, BTNX-4, BTNX-5, BTNX-6, BTNX-7, BTNX-8, BTNX-9, MCU1-MCU3_GPIO, RST_2560
- net labels removed: 3.3V, 5V, MCU1_LED_CTRL, MIDI_IN, MIDI_OUT, SCL, SDA, button-01, button-02, button-03, button-04, button-05, button-06, button-07, button-08, button-09, button-10, button-11, button-12, button-13, button-14, button-15, button-16, button-17, button-18, button-19, button-20, button-21, button-22, button-23, button-24, button-25, button-26, button-27, button-28, button-29, button-30, button-31, button-32, button-33, button-34, button-35, button-36, button-37, button-38, button-39, button-40, button-41, button-42, button-43, button-44, button-45, button-46, button-47, button-48, button-49, button-50, button-51, button-52, button-53, button-54, button-55, button-56, button-57, button-58, button-59, button-60, button-61, button-X-1, button-X-10, button-X-11, button-X-12, button-X-2, button-X-3, button-X-4, button-X-5, button-X-6, button-X-7, button-X-8, button-X-9
- wire segments 525 -> 639
- no-connect marks 7 -> 5
Other:
- note added: "12V 2A"
- note added: "512 B RAM\n73 LEDs = 73x3 = 219B needed to store all LEDs"
- note added: "AIN3"
- note added: "Buttons 1-4"
- note added: "Buttons 5-61"
- note added: "Buttons X1-X12"
- note added: "Choose one or the other to drive the LED,\nSPI MOSI, or Output Compare"
- note added: "DNP options in case you want \nto experiment with running LEDs from\nArudino front-end"
- note added: "Diode Protects in case\nData present without Power"
- note added: "Extra HW for sharing button input"
- note added: "GPIO/USART1_XCK"
- note added: "HW Changes:"
- note added: "OC0/OC1"
- note added: "PCB MOUNT\nMETA BUTTONS"
- note added: "PROG_CTRL_1 HIGH: Shorts pin 5 - 6 (DFU MODE)\nPROG_CTRL_2 HIGH: Shorts pin 4 - 6 (ARDUINO MODE)\n_1 & _2 LOW: USB Midi Mode"
- note added: "Program over ICSP.\n No Arudino interface, only acts as Meta-Button control (MCU programming mode), \n& LED driving interface"
- note added: "QUESTION, DO WE NEED RESET BUTTONS ON BOARD?\n"
- note added: "QUESTION,\nTIE SHIELD TO GND?\nTODO, FIGURE OUT.\nTODO, SMD OPTO"
- note added: "RESET\nCONTROL"
- note added: "Spare"
- note added: "TODO:\nI'm not sure ESD protection here is right,\nwhat exactly is softpot? \n\nQUESTION:potentiometer INPUT or simulated potentiometer output???"
- note added: "Todo FOOTPRINTS"
- note added: "USART1 RX"
- note added: "\nButton 37 Remapped from PH1 to PH7\nButton 60 Remapped from PF0 to PBO"
- note removed: "META BUTTONS"
- note removed: "QUESTION, DO WE NEED RESET BUTTONS ON BOARD?\nTODO, ADD"
- note removed: "QUESTION,\nADC OR GPIO FOR THIS?\nEITHER WORKS, \nADC WILL REQUIRE MOVING SOME BUTTONS"
- note removed: "QUESTION,\nTIE SHIELD TO GND?\nTODO, FIGURE OUT"
- note removed: "TODO"
- note removed: "TODO FIND A XTAL/RESONATOR THAT CAN DO BOTH MCUS ??"
- note removed: "TODO, HOOK THESE UP FOR PROGRAMMING CONTROL\nTODO, DESIGN FET/RELAY CIRCUIT\n(REPLACES JUMPERS)"
- note removed: "TODO, IS DIODE TO 5V ON RESET NEEDED?!??"
- note removed: "TODO, JUMPER JP5: PB4-7"
- note removed: "TODO,\nCAN PROBABLY GET AWAY WITHOUT OSCILLATOR HERE,\nDOUBLE CHECK ACCURACY"
- note removed: "TODO,\nRESET_EN JUMPER??"
- note removed: "TODO\nFIGURE OUT IF UVCC IS CORRECTLY SETUP HERE"
- note removed: "TODO\nUGND/PAD/GND GNDS AND JUMPERS ARE WEIRD ON MEGA??"
- moved on the sheet: C16, C17, C18, C2, C20, C23, C33, C34, C35, C36, C37, C38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

Commit message: Schematic review
- Updates blocks
- Removes RGB LEDS from off board
- Fixes ERC errors
Parts:
- C16, C17: value 22PF -> 22pF
- Y3: value 16MHz CSTNE16M0V530000R0 -> 16MHz
Connections:
- no-connect marks 5 -> 9
Other:
- note added: "BARREL POWER DETECT"
- note added: "MCU FILTER"
- note added: "NO LEDs"
- note added: "RESET CONTROL"
- note added: "SPARE"
- note removed: "50mA each LED, \nx12 = 600mA minimum"
- note removed: "BARREL POWER \nDETECT"
- note removed: "HW Changes:"
- note removed: "RESET\nCONTROL"
- note removed: "Spare"
- note removed: "\nButton 37 Remapped from PH1 to PH7\nButton 60 Remapped from PF0 to PBO"
- moved on the sheet: C1, C10, C11, C12, C13, C14, C15, C16, C17, C18, C19, C2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

Commit message: Minor schematic and library changes
Fixes some typos; changes oscillators to be common to all MCUs; SMD for MIDI opto input
Parts:
- removed C16, C17: 22pF, Capacitor_SMD:C_0603_1608Metric, symbol Device:C
- removed C34, C35: 22PF, Capacitor_SMD:C_0603_1608Metric, symbol Device:C
- removed C39, C4, C41: 100nf, Capacitor_SMD:C_0603_1608Metric, symbol Device:C
- removed R21: 4.7k, Resistor_SMD:R_0603_1608Metric, symbol Device:R
- removed U3: 6N138, symbol Isolator:6N138
- removed Y1, Y2: Crystal, Crystal:Crystal_HC49-U_Vertical, symbol Device:Crystal
- added C? (x6): 1uF 25V, Capacitor_SMD:C_0805_2012Metric, symbol lib_symbol:C
- added C? (x5): 100nf, Capacitor_SMD:C_0603_1608Metric, symbol Device:C
- added C? (x2): DNP-1uF 25V, Capacitor_SMD:C_0805_2012Metric, symbol lib_symbol:C
- added R?: 19.1k, Resistor_SMD:R_0603_1608Metric, symbol Device:R
- added U?: 6N137, symbol lib_symbol:6N137
- added Y? (x2): 16MHz, Crystal:Resonator_SMD_muRata_CSTxExxV-3Pin_3.0x1.1mm, symbol Device:Resonator
Connections:
- net Earth is gone; now on net GND: D16.3 (A), D2.3 (A), D3.3 (A)
- net 5VA_MCU: now also C?.1
- net 5V_MCU: now also R28.1, C?.1, C?.1, C?.1, C?.1, R?.1, U?.7 (EN), U?.8 (VCC); no longer R28.2
- net 5V_USB: now also C?.1, C?.1, C?.1, C?.1
- net AREF: now also C?.1
- net GND: now also C?.2, C?.2, C?.2, C?.2, C?.2, C?.2, C?.2, C?.2, C?.2, C?.2, C?.2, C?.2, C?.2, U?.5 (GND), Y?.2, Y?.2
- net MCU2_RST: now also C?.1, R?.2; no longer C33.1, R28.1
- net MCU3_RST: now also C33.1, R28.2
- net at D13.2 (K), R17.1: now also U?.2 (A)
- net at D13.3 (A), J6.5: now also U?.3 (C)
- net at R23.1, U4.5: now also U?.6 (VO)
- net at J6.2: now also C?.1
- net at U5.1 (XTAL1): now also Y?.1
- net at U5.2 (PC0/XTAL2): now also Y?.3
- net at U2.1 (XTAL1): now also Y?.1
- net at U2.2 (PC0/XTAL2): now also Y?.3
- net SHIELD: no longer names the net of J6.S1 (SHIELD), J6.S2 (SHIELD)
- net SHIELD: now also C?.1
- no-connect marks 9 -> 8
Other:
- note added: "ARDUINO INTERFACE MCU (2)"
- note added: "FOOTPRINT NOTE\n"
- note added: "LED CONTROLLER MCU (3)"
- note added: "MAIN MCU (1)"
- note added: "NONSTANDARD SO-8 PACKAGE"
- note added: "Placement Notes:\nPlace MLCC near MCU pins"
- note removed: "ARDUINO INTERFACE MCU"
- note removed: "LED CONTROLLER MCU"
- note removed: "MAIN MCU"
- note removed: "QUESTION,\nTIE SHIELD TO GND?\nTODO, FIGURE OUT.\nTODO, SMD OPTO"
- note removed: "TODO: CONFIRM I TRANSFERRED THIS BLOCK CORRECTLY"
- moved on the sheet: C28, C31
