File: rainboard-pcb/kicad_proj/rainboard_newfighter/rainboard_newfighter.sch (KiCad schematic (older format))
At the start: 171 parts, among them J1 54-00167, J10 Conn_01x02_Female, J11 Conn_01x02_Female, J12 Conn_01x02_Female, J13 Conn_01x02_Female, J14 Conn_01x02_Female, J15 SDS-50J, J16 Conn_01x02_Female, J17 PH2-06-UA, J18 Conn_01x03, J19 Conn_01x03, J2 SDS-50J, J20 PH2-06-UA, J21 PH2-06-UA, J3 USB_B, J4 Conn_01x02_Female, J5 Conn_01x02_Female, J6 Conn_01x02_Female, J7 Conn_01x02_Female, J8 Conn_01x02_Female, J9 Conn_01x02_Female, Q2 DUAL 30V NMOS, Q3 DUAL 30V NMOS, U1 6N137, U3 74HC14, U4 ATmega16U2-MU, U5 ATmega16U2-MU, U6 ATmega2560-16AU, Y1 16MHz, Y2 16MHz, Y3 16MHz

Commit message: Modified electrolytics and setup board for layout
Parts:
- removed D6: 12Vw, Diode_SMD:D_SMA, symbol lib_symbol:D_Zener
- added D6: 6V, rainboard_fp:SOT23-3, symbol lib_symbol:D_Zener_SOT23
- C15, C19, C42: value 470uF 25V -> 470uF 10V; footprint Capacitor_SMD:CP_Elec_10x10 -> Capacitor_SMD:CP_Elec_6.3x7.7
- D1: PN (none) -> DLP05LC-7-F
Connections:
- net 5V_WALL: now also D6.3 (NC)
- net GND: now also D6.1 (K), D6.2 (A)
Changed lines of the file:
@@
 	2000 1350 2450 1350
 $Comp
-L lib_symbol:D_Zener D6
-U 1 1 6038EFA9
-P 4850 1700
-F 0 "D6" H 4850 1800 50  0000 C CNN
-F 1 "12Vw " H 4850 1600 50  0000 C CNN
-F 2 "Diode_SMD:D_SMA" H 4850 1700 50  0001 C CNN
-F 3 "~" H 4850 1700 50  0001 C CNN
-F 4 "SMAJ12A" H 4850 1900 50  0001 C CNN "PN"
-	1    4850 1700
-	0    1    1    0
-$EndComp
-$Comp
 L lib_symbol:Polyfuse F1
 U 1 1 603A141D
@@
 P 5550 1650
 F 0 "C15" H 5575 1750 50  0000 L CNN
-F 1 "470uF 25V" H 5575 1550 50  0000 L CNN
-F 2 "Capacitor_SMD:CP_Elec_10x10" H 5588 1500 50  0001 C CNN
+F 1 "470uF 10V" H 5575 1550 50  0000 L CNN
+F 2 "Capacitor_SMD:CP_Elec_6.3x7.7" H 5588 1500 50  0001 C CNN
 F 3 "~" H 5550 1650 50  0001 C CNN
 F 4 "UCW1E471MNL1GS" V 5400 1600 50  0001 C CNN "PN"
@@
 P 8650 4450
 F 0 "C19" H 8675 4550 50  0000 L CNN
-F 1 "470uF 25V" H 8675 4350 50  0000 L CNN
-F 2 "Capacitor_SMD:CP_Elec_10x10" H 8688 4300 50  0001 C CNN
+F 1 "470uF 10V" H 8675 4350 50  0000 L CNN
+F 2 "Capacitor_SMD:CP_Elec_6.3x7.7" H 8688 4300 50  0001 C CNN
 F 3 "~" H 8650 4450 50  0001 C CNN
 F 4 "UCW1E471MNL1GS" V 8450 4250 50  0001 C CNN "PN"
@@
 P 23650 2000
 F 0 "C42" H 23675 2100 50  0000 L CNN
-F 1 "470uF 25V" H 23675 1900 50  0000 L CNN
-F 2 "Capacitor_SMD:CP_Elec_10x10" H 23688 1850 50  0001 C CNN
+F 1 "470uF 10V" H 23675 1900 50  0000 L CNN
+F 2 "Capacitor_SMD:CP_Elec_6.3x7.7" H 23688 1850 50  0001 C CNN
 F 3 "~" H 23650 2000 50  0001 C CNN
 F 4 "UCW1E471MNL1GS" V 23800 1400 50  0001 C CNN "PN"
@@
 F 2 "rainboard_fp:SOT23-3" H 2000 1700 50  0001 C CNN
 F 3 "~" H 2000 1700 50  0001 C CNN
+F 4 "DLP05LC-7-F" V 2000 1700 50  0001 C CNN "PN"
 	1    2000 1700
 	0    1    1    0
@@
 $EndComp
 Connection ~ 6150 850
+$Comp
+L lib_symbol:D_Zener_SOT23 D6
+U 1 1 62B334D3
+P 4850 1700
+F 0 "D6" V 4804 1780 50  0000 L CNN
+F 1 "6V" V 4895 1780 50  0000 L CNN
+F 2 "rainboard_fp:SOT23-3" H 4850 1700 50  0001 C CNN
+F 3 "~" H 4850 1700 50  0001 C CNN
+F 4 "DLP05LC-7-F" V 4850 1700 50  0001 C CNN "PN"
+	1    4850 1700
+	0    1    1    0
+$EndComp
 $EndSCHEMATC

Commit message: Forgot to update electrolytic PN
Parts:
- C15, C19, C42: PN UCW1E471MNL1GS -> EEE-FTA471XAP
Changed lines of the file:
@@
 F 2 "Capacitor_SMD:CP_Elec_6.3x7.7" H 5588 1500 50  0001 C CNN
 F 3 "~" H 5550 1650 50  0001 C CNN
-F 4 "UCW1E471MNL1GS" V 5400 1600 50  0001 C CNN "PN"
+F 4 "EEE-FTA471XAP" V 5400 1600 50  0001 C CNN "PN"
 	1    5550 1650
 	1    0    0    -1
@@
 F 2 "Capacitor_SMD:CP_Elec_6.3x7.7" H 8688 4300 50  0001 C CNN
 F 3 "~" H 8650 4450 50  0001 C CNN
-F 4 "UCW1E471MNL1GS" V 8450 4250 50  0001 C CNN "PN"
+F 4 "EEE-FTA471XAP" V 8450 4250 50  0001 C CNN "PN"
 	1    8650 4450
 	1    0    0    -1
@@
 F 2 "Capacitor_SMD:CP_Elec_6.3x7.7" H 23688 1850 50  0001 C CNN
 F 3 "~" H 23650 2000 50  0001 C CNN
-F 4 "UCW1E471MNL1GS" V 23800 1400 50  0001 C CNN "PN"
+F 4 "EEE-FTA471XAP" V 23800 1400 50  0001 C CNN "PN"
 	1    23650 2000
 	1    0    0    -1
