File: rainboard-pcb/kicad_proj/rainboard_newfighter/rainboard_newfighter.sch (KiCad schematic (older format))
At the start: 171 parts, among them J1 54-00167, J10 Conn_01x02_Female, J11 Conn_01x02_Female, J12 Conn_01x02_Female, J13 Conn_01x02_Female, J14 Conn_01x02_Female, J15 SDS-50J, J16 Conn_01x02_Female, J17 PH2-06-UA, J18 Conn_01x03, J19 Conn_01x03, J2 SDS-50J, J20 PH2-06-UA, J21 PH2-06-UA, J3 USB_B, J4 Conn_01x02_Female, J5 Conn_01x02_Female, J6 Conn_01x02_Female, J7 Conn_01x02_Female, J8 Conn_01x02_Female, J9 Conn_01x02_Female, Q2 DUAL 30V NMOS, Q3 DUAL 30V NMOS, U1 6N137, U3 74HC14, U4 ATmega16U2-MU, U5 ATmega16U2-MU, U6 ATmega2560-16AU, Y1 16MHz, Y2 16MHz, Y3 16MHz

Commit message: Moves meta button connectors to correct spots
Updates locations for layout to continue
Parts:
- C1, C11, C2: footprint Capacitor_SMD:C_0805_2012Metric -> (none)
- D3: footprint Package_TO_SOT_SMD:SOT-23 -> (none)
- J2: footprint rainboard_fp:CUI_SDS-50J -> (none)
- R1, R8: footprint Resistor_SMD:R_0805_2012Metric -> (none)
- R4: footprint Resistor_SMD:R_0603_1608Metric -> (none)
- U1: footprint rainboard_fp:COUPL_6N138SDM -> (none)
Connections:
- net GND: now also U3.5, U3.9
- net at R8.1, U1.6 (VO): no longer U3.5
- net at U3.6: no longer U3.9
- net MIDI-IN: no longer names the net of U3.8
- net MIDI-IN: no longer U6.45 (PD2)
- no-connect marks 7 -> 10
Other:
- note added: "MIDI IN NOT USED, STILL\nON SCHEMATIC AS A \nREFERENCE"
- note removed: "FOOTPRINT NOTE\n"
- note removed: "NONSTANDARD SO-8 PACKAGE"
- moved on the sheet: C18, D15, R14

Commit message: Review and gerber export of v1a
Parts:
- removed JP4, JP5: Jumper, Jumper:SolderJumper-2_P1.3mm_Bridged_Pad1.0x1.5mm, symbol lib_symbol:Jumper
- J18, J19: footprint Connector_JST:JST_XH_B3B-XH-AM_1x03_P2.50mm_Vertical -> rainboard_fp:009296003202906
Connections:
- net GNDA is gone; now on net GND: C29.2, R35.2, R36.2, R38.2
- net GND: now also U6.11 (GND), U6.32 (GND), U6.62 (GND), U6.81 (GND), U6.99 (GND)
