File: rainboard-pcb/kicad_proj/rainboard_newfighter/MetaButton.sch (KiCad schematic (older format))
At the start: 7 parts, among them SW13 SANWA-OBSF24

Commit message: Removed RGB from buttons, part numbers updated, cleaned up schematic
Parts:
- C84: PN (none) -> CC0603KRX7R9BB104
- D31: PN (none) -> WS2812B
- R58: PN (none) -> RC0603FR-07210RL
- R59: PN (none) -> RC0603JR-074K7L
- R60, R61: PN (none) -> RC0603FR-0719K1L
Changed lines of the file:
@@
 $Descr A4 11693 8268
 encoding utf-8
-Sheet 16 65
+Sheet 5 65
 Title ""
 Date ""
@@
 AR Path="/601692FD/602ABA7A/601BA75D" Ref="SW15"  Part="1"
 AR Path="/601692FD/602ABA92/601BA75D" Ref="SW16"  Part="1"
-F 0 "SW16" H 3900 2500 50  0000 C CNN
+F 0 "SW15" H 3900 2500 50  0000 C CNN
 F 1 "SANWA-OBSF24" H 3900 2540 50  0001 C CNN
 F 2 "" H 3900 2800 50  0001 C CNN
@@
 AR Path="/601692FD/602ABA7A/601BA763" Ref="D33"  Part="1"
 AR Path="/601692FD/602ABA92/601BA763" Ref="D34"  Part="1"
-F 0 "D34" H 1700 2075 50  0000 R BNN
+F 0 "D33" H 1700 2075 50  0000 R BNN
 F 1 "WS2812B" H 1550 1625 50  0000 L TNN
 F 2 "LED_SMD:LED_WS2812B_PLCC4_5.0x5.0mm_P3.2mm" H 1550 1550 50  0001 L TNN
 F 3 "https://cdn-shop.adafruit.com/datasheets/WS2812B.pdf" H 1600 1475 50  0001 L TNN
+F 4 "WS2812B" H 1500 1850 50  0001 C CNN "PN"
 	1    1500 1850
 	1    0    0    -1
@@
 AR Path="/601692FD/602ABA7A/601BA769" Ref="#PWR0213"  Part="1"
 AR Path="/601692FD/602ABA92/601BA769" Ref="#PWR0216"  Part="1"
-F 0 "#PWR0216" H 3900 2650 50  0001 C CNN
+F 0 "#PWR0213" H 3900 2650 50  0001 C CNN
 F 1 "GND" H 3900 2750 50  0000 C CNN
 F 2 "" H 3900 2900 50  0001 C CNN
@@
 AR Path="/601692FD/602ABA7A/601BA76F" Ref="#PWR0214"  Part="1"
 AR Path="/601692FD/602ABA92/601BA76F" Ref="#PWR0217"  Part="1"
-F 0 "#PWR0217" H 1500 2000 50  0001 C CNN
+F 0 "#PWR0214" H 1500 2000 50  0001 C CNN
 F 1 "GND" H 1500 2100 50  0000 C CNN
 F 2 "" H 1500 2250 50  0001 C CNN
@@
 AR Path="/601692FD/602ABA7A/601BA77D" Ref="R66"  Part="1"
 AR Path="/601692FD/602ABA92/601BA77D" Ref="R70"  Part="1"
-F 0 "R70" V 2100 1800 50  0000 L CNN
+F 0 "R66" V 2100 1800 50  0000 L CNN
 F 1 "210R" V 1900 1800 50  0000 L CNN
 F 2 "Resistor_SMD:R_0805_2012Metric" V 1930 1850 50  0001 C CNN
 F 3 "~" H 2000 1850 50  0001 C CNN
 F 4 "C228630" H 2000 1850 50  0001 C CNN "LCSC"
+F 5 "RC0603FR-07210RL" H 2000 1850 50  0001 C CNN "PN"
 	1    2000 1850
 	0    1    1    0
@@
 AR Path="/601692FD/602ABA7A/601BA78A" Ref="C86"  Part="1"
 AR Path="/601692FD/602ABA92/601BA78A" Ref="C87"  Part="1"
-F 0 "C87" H 2750 1650 50  0000 L CNN
+F 0 "C86" H 2750 1650 50  0000 L CNN
 F 1 "100nf" V 3000 1650 50  0000 L CNN
 F 2 "Capacitor_SMD:C_0603_1608Metric" H 2888 1650 50  0001 C CNN
 F 3 "~" H 2850 1800 50  0001 C CNN
 F 4 "C14663" H 2850 1800 50  0001 C CNN "LCSC"
+F 5 "CC0603KRX7R9BB104" H 2850 1800 50  0001 C CNN "PN"
 	1    2850 1800
 	1    0    0    -1
@@
 AR Path="/601692FD/602ABA7A/601BA792" Ref="#PWR0215"  Part="1"
 AR Path="/601692FD/602ABA92/601BA792" Ref="#PWR0218"  Part="1"
-F 0 "#PWR0218" H 2850 1800 50  0001 C CNN
+F 0 "#PWR0215" H 2850 1800 50  0001 C CNN
 F 1 "GND" H 2850 1900 50  0000 C CNN
 F 2 "" H 2850 2050 50  0001 C CNN
@@
 AR Path="/601692FD/602ABA7A/6027B05D" Ref="R67"  Part="1"
 AR Path="/601692FD/602ABA92/6027B05D" Ref="R71"  Part="1"
-F 0 "R71" H 3720 1796 50  0000 L CNN
+F 0 "R67" H 3720 1796 50  0000 L CNN
 F 1 "4.7k" H 3720 1705 50  0000 L CNN
 F 2 "Resistor_SMD:R_0603_1608Metric" V 3580 1750 50  0001 C CNN
 F 3 "~" H 3650 1750 50  0001 C CNN
 F 4 "C23162" H 3650 1750 50  0001 C CNN "LCSC"
+F 5 "RC0603JR-074K7L" H 3650 1750 50  0001 C CNN "PN"
 	1    3650 1750
 	1    0    0    -1
@@
 AR Path="/601692FD/602ABA7A/6027B064" Ref="R68"  Part="1"
 AR Path="/601692FD/602ABA92/6027B064" Ref="R72"  Part="1"
-F 0 "R72" V 4150 1900 50  0000 L CNN
+F 0 "R68" V 4150 1900 50  0000 L CNN
 F 1 "19.1k" V 4050 1850 50  0000 L CNN
 F 2 "Resistor_SMD:R_0603_1608Metric" V 4180 1950 50  0001 C CNN
 F 3 "~" H 4250 1950 50  0001 C CNN
 F 4 "C22897" H 4250 1950 50  0001 C CNN "LCSC"
+F 5 "RC0603FR-0719K1L" H 4250 1950 50  0001 C CNN "PN"
 	1    4250 1950
 	0    1    1    0
@@
 AR Path="/601692FD/602ABA7A/602835D9" Ref="R69"  Part="1"
 AR Path="/601692FD/602ABA92/602835D9" Ref="R73"  Part="1"
-F 0 "R73" V 4250 2200 50  0000 L CNN
+F 0 "R69" V 4250 2200 50  0000 L CNN
 F 1 "19.1k" V 4150 2150 50  0000 L CNN
 F 2 "Resistor_SMD:R_0603_1608Metric" V 4280 2250 50  0001 C CNN
 F 3 "~" H 4350 2250 50  0001 C CNN
 F 4 "C22897" H 4350 2250 50  0001 C CNN "LCSC"
+F 5 "RC0603FR-0719K1L" H 4350 2250 50  0001 C CNN "PN"
 	1    4350 2250
 	0    1    1    0
