File: rainboard-pcb/kicad_proj/rainboard_newfighter/rainboard_newfighter.kicad_pcb (KiCad board)
At the start: 2 copper layers, 260 x 253.6 mm, 498 parts, among them J1 EJ508A, J10 Conn_01x02_Female, J11 Conn_01x02_Female, J12 Conn_01x02_Female, J13 Conn_01x02_Female, J14 Conn_01x02_Female, J15 Conn_01x02_Female, J16 Conn_01x02_Female, J17 Conn_01x02_Female, J18 Conn_01x02_Female, J19 Conn_01x02_Female, J2 USB_B, J20 Conn_01x02_Female, J21 Conn_01x02_Female, J3 Conn_01x03, J4 Conn_01x03, J5 PH2-06-UA, J6 SDS-50J, J7 SDS-50J, J8 PH2-06-UA, J9 PH2-06-UA, Q1 DUAL 30V NMOS, Q2 DUAL 30V NMOS, Q3 30V 10mOhm, SW1 SANWA-OBSF24, SW10 SANWA-OBSF24, SW11 SANWA-OBSF24, SW12 SANWA-OBSF24, SW13 SANWA-OBSF24, SW14 SANWA-OBSF24, SW15 SANWA-OBSF24, SW16 SANWA-OBSF24, SW17 SANWA-OBSF24, SW18 SANWA-OBSF24, SW19 SANWA-OBSF24, SW2 SANWA-OBSF24, SW20 SANWA-OBSF24, SW21 SANWA-OBSF24, SW22 SANWA-OBSF24, SW23 SANWA-OBSF24, SW24 SANWA-OBSF24, SW25 SANWA-OBSF24, SW26 SANWA-OBSF24, SW27 SANWA-OBSF24, SW28 SANWA-OBSF24, SW29 SANWA-OBSF24, SW3 SANWA-OBSF24, SW30 SANWA-OBSF24, SW31 SANWA-OBSF24, SW32 SANWA-OBSF24, SW33 SANWA-OBSF24, SW34 SANWA-OBSF24, SW35 SANWA-OBSF24, SW36 SANWA-OBSF24, SW37 SANWA-OBSF24, SW38 SANWA-OBSF24, SW39 SANWA-OBSF24, SW4 SANWA-OBSF24, SW40 SANWA-OBSF24, SW41 SANWA-OBSF24, SW42 SANWA-OBSF24, SW43 SANWA-OBSF24, SW44 SANWA-OBSF24, SW45 SANWA-OBSF24, SW46 SANWA-OBSF24, SW47 SANWA-OBSF24, SW48 SANWA-OBSF24, SW49 SANWA-OBSF24, SW5 SANWA-OBSF24, SW50 SANWA-OBSF24, SW51 SANWA-OBSF24, SW52 SANWA-OBSF24, SW53 SANWA-OBSF24, SW54 SANWA-OBSF24, SW55 SANWA-OBSF24, SW56 SANWA-OBSF24, SW57 SANWA-OBSF24, SW58 SANWA-OBSF24, SW59 SANWA-OBSF24, SW6 SANWA-OBSF24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

Commit message: Moves meta buttons to correct config, adds back on board buttons.
Parts:
- removed C126, C127, C128, C129, C130, C131, C132, C133, C134, C135, C136, C137, C138, C139, C140, C141, C142, C143, C144, C145, C146, C147, C148, C149, C150, C151, C152, C153, C154, C155, C156, C157, C158: 100nf, Capacitor_SMD:C_0603_1608Metric
- removed D80, D81, D82, D83, D84, D85, D86, D87, D88, D89, D90, D91: WS2812B, LED_SMD:LED_WS2812B_PLCC4_5.0x5.0mm_P3.2mm
- removed R175, R176, R177, R178, R179, R180, R181, R182, R183, R184, R185, R186, R187: 210R, Resistor_SMD:R_0805_2012Metric
- added C51: 470uF 25V, Capacitor_SMD:CP_Elec_10x10, F.Cu at (167.1, 24.7)
- added C52: 470uF 25V, Capacitor_SMD:CP_Elec_10x10, F.Cu at (167.1, 36.6)
- added C53: 470uF 25V, Capacitor_SMD:CP_Elec_10x10, F.Cu at (181.1, 24.7)
- added C54: 470uF 25V, Capacitor_SMD:CP_Elec_10x10, F.Cu at (181.1, 36.6)
- added C55: 10uF 25V, Capacitor_SMD:C_1206_3216Metric, F.Cu at (196.3, 23.8)
- added C56: 10uF 25V, Capacitor_SMD:C_1206_3216Metric, F.Cu at (190.7, 20.5)
- added C57: 10uF 25V, Capacitor_SMD:C_1206_3216Metric, F.Cu at (162.6, 47.5)
- added C58: 10uF 25V, Capacitor_SMD:C_1206_3216Metric, F.Cu at (168.2, 44.2)
- added C59: 10uF 25V, Capacitor_SMD:C_1206_3216Metric, F.Cu at (168.2, 47.5)
- added C60: 10uF 25V, Capacitor_SMD:C_1206_3216Metric, F.Cu at (196.3, 20.5)
- added C61: 10uF 25V, Capacitor_SMD:C_1206_3216Metric, F.Cu at (190.7, 23.8)
- added C62: 10uF 25V, Capacitor_SMD:C_1206_3216Metric, F.Cu at (190.7, 27.0)
- added C63: 10uF 25V, Capacitor_SMD:C_1206_3216Metric, F.Cu at (201.9, 20.5)
- added C64: 10uF 25V, Capacitor_SMD:C_1206_3216Metric, F.Cu at (162.6, 44.2)
- added C65: 100nf, Capacitor_SMD:C_0603_1608Metric, F.Cu at (218.2, 59.4)
- added C66: 100nf, Capacitor_SMD:C_0603_1608Metric, F.Cu at (264.5, 23.0)
- added C67: 100nf, Capacitor_SMD:C_0603_1608Metric, F.Cu at (308.6, -16.2)
- added C68: 100nf, Capacitor_SMD:C_0603_1608Metric, F.Cu at (248.5, 43.7)
- added C69: 100nf, Capacitor_SMD:C_0603_1608Metric, F.Cu at (264.5, 33.3)
- added C70: 100nf, Capacitor_SMD:C_0603_1608Metric, F.Cu at (292.6, 4.43)
- added C71: 100nf, Capacitor_SMD:C_0603_1608Metric, F.Cu at (234.3, 54.0)
- added C72: 100nf, Capacitor_SMD:C_0603_1608Metric, F.Cu at (280.5, 23.0)
- added C73: 100nf, Capacitor_SMD:C_0603_1608Metric, F.Cu at (308.6, -5.89)
- added C74: 100nf, Capacitor_SMD:C_0603_1608Metric, F.Cu at (324.7, -26.5)
- added C75: 100nf, Capacitor_SMD:C_0603_1608Metric, F.Cu at (340.7, -36.9)
- added C76: 100nf, Capacitor_SMD:C_0603_1608Metric, F.Cu at (248.5, 33.3)
- added C77: 100nf, Capacitor_SMD:C_0603_1608Metric, F.Cu at (324.7, -16.2)
- added C78: 100nf, Capacitor_SMD:C_0603_1608Metric, F.Cu at (250.3, 54.0)
- added C79: 100nf, Capacitor_SMD:C_0603_1608Metric, F.Cu at (264.5, 43.7)
- added C80: 100nf, Capacitor_SMD:C_0603_1608Metric, F.Cu at (280.5, 33.3)
- added C81: 100nf, Capacitor_SMD:C_0603_1608Metric, F.Cu at (308.6, 4.43)
- added C82: 100nf, Capacitor_SMD:C_0603_1608Metric, F.Cu at (296.5, 14.8)
- added C83: 100nf, Capacitor_SMD:C_0603_1608Metric, F.Cu at (324.7, -5.89)
- added C84: 100nf, Capacitor_SMD:C_0603_1608Metric, F.Cu at (340.7, -26.5)
- added C85: 100nf, Capacitor_SMD:C_0603_1608Metric, F.Cu at (356.7, -36.9)
- added C86: 100nf, Capacitor_SMD:C_0603_1608Metric, F.Cu at (340.7, -16.2)
- added C87: 100nf, Capacitor_SMD:C_0603_1608Metric, F.Cu at (296.5, 25.1)
- added D19: WS2812B, LED_SMD:LED_WS2812B_PLCC4_5.0x5.0mm_P3.2mm, F.Cu at (212.0, 58.5)
- added D20: WS2812B, LED_SMD:LED_WS2812B_PLCC4_5.0x5.0mm_P3.2mm, F.Cu at (258.3, 22.1)
- added D21: WS2812B, LED_SMD:LED_WS2812B_PLCC4_5.0x5.0mm_P3.2mm, F.Cu at (302.4, -17.1)
- added D22: WS2812B, LED_SMD:LED_WS2812B_PLCC4_5.0x5.0mm_P3.2mm, F.Cu at (242.2, 42.8)
- added D23: WS2812B, LED_SMD:LED_WS2812B_PLCC4_5.0x5.0mm_P3.2mm, F.Cu at (258.3, 32.4)
- added D24: WS2812B, LED_SMD:LED_WS2812B_PLCC4_5.0x5.0mm_P3.2mm, F.Cu at (286.4, 3.54)
- added D25: WS2812B, LED_SMD:LED_WS2812B_PLCC4_5.0x5.0mm_P3.2mm, F.Cu at (228.0, 53.1)
- added D26: WS2812B, LED_SMD:LED_WS2812B_PLCC4_5.0x5.0mm_P3.2mm, F.Cu at (274.3, 22.1)
- added D27: WS2812B, LED_SMD:LED_WS2812B_PLCC4_5.0x5.0mm_P3.2mm, F.Cu at (302.4, -6.79)
- added D28: WS2812B, LED_SMD:LED_WS2812B_PLCC4_5.0x5.0mm_P3.2mm, F.Cu at (318.4, -27.4)
- added D29: WS2812B, LED_SMD:LED_WS2812B_PLCC4_5.0x5.0mm_P3.2mm, F.Cu at (334.5, -37.7)
- added D30: WS2812B, LED_SMD:LED_WS2812B_PLCC4_5.0x5.0mm_P3.2mm, F.Cu at (242.2, 32.4)
- added D31: WS2812B, LED_SMD:LED_WS2812B_PLCC4_5.0x5.0mm_P3.2mm, F.Cu at (318.4, -17.1)
- added D32: WS2812B, LED_SMD:LED_WS2812B_PLCC4_5.0x5.0mm_P3.2mm, F.Cu at (244.1, 53.1)
- added D33: WS2812B, LED_SMD:LED_WS2812B_PLCC4_5.0x5.0mm_P3.2mm, F.Cu at (258.3, 42.8)
- added D34: WS2812B, LED_SMD:LED_WS2812B_PLCC4_5.0x5.0mm_P3.2mm, F.Cu at (274.3, 32.4)
- added R54: 210R, Resistor_SMD:R_0805_2012Metric, F.Cu at (199.6, 41.6)
- added R55: 210R, Resistor_SMD:R_0805_2012Metric, F.Cu at (192.8, 47.9)
- added R56: 210R, Resistor_SMD:R_0805_2012Metric, F.Cu at (207.8, 35.4)
- added R57: 210R, Resistor_SMD:R_0805_2012Metric, F.Cu at (212.2, 32.4)
- added R58: 210R, Resistor_SMD:R_0805_2012Metric, F.Cu at (212.2, 29.5)
- added R59: 210R, Resistor_SMD:R_0805_2012Metric, F.Cu at (203.3, 29.8)
- added R60: 210R, Resistor_SMD:R_0805_2012Metric, F.Cu at (190.8, 44.9)
- added R61: 210R, Resistor_SMD:R_0805_2012Metric, F.Cu at (203.3, 32.8)
- added R62: 210R, Resistor_SMD:R_0805_2012Metric, F.Cu at (209.0, 26.5)
- added R63: 210R, Resistor_SMD:R_0805_2012Metric, F.Cu at (190.8, 42.0)
- added R64: 210R, Resistor_SMD:R_0805_2012Metric, F.Cu at (198.9, 35.7)
- added R65: 210R, Resistor_SMD:R_0805_2012Metric, F.Cu at (215.8, 20.3)
- added R66: 210R, Resistor_SMD:R_0805_2012Metric, F.Cu at (184.0, 49.9)
- added R67: 210R, Resistor_SMD:R_0805_2012Metric, F.Cu at (199.6, 44.6)
- added R68: 210R, Resistor_SMD:R_0805_2012Metric, F.Cu at (195.2, 42.0)
- added R69: 210R, Resistor_SMD:R_0805_2012Metric, F.Cu at (198.9, 38.7)
- added R70: 210R, Resistor_SMD:R_0805_2012Metric, F.Cu at (207.8, 29.5)
- added R71: 210R, Resistor_SMD:R_0805_2012Metric, F.Cu at (188.4, 49.9)
- added R72: 210R, Resistor_SMD:R_0805_2012Metric, F.Cu at (207.8, 32.4)
- added R73: 210R, Resistor_SMD:R_0805_2012Metric, F.Cu at (194.5, 39.0)
- C1: value 10uF 25V -> DNP-1uF 25V; footprint Capacitor_SMD:C_1206_3216Metric -> Capacitor_SMD:C_0805_2012Metric
- C100, C101, C30, C92, C93, C94, C95, C96, C97, C98, C99: value 10uF 25V -> 100nf; footprint Capacitor_SMD:C_1206_3216Metric -> Capacitor_SMD:C_0603_1608Metric
- C12, C31, C33, C43, C47: value 100nf -> 1uF 25V; footprint Capacitor_SMD:C_0603_1608Metric -> Capacitor_SMD:C_0805_2012Metric
- C13, C18, C34, C45, C50: value 1uF 25V -> 100nf; footprint Capacitor_SMD:C_0805_2012Metric -> Capacitor_SMD:C_0603_1608Metric
- C14, C20, C38: value 470uF 25V -> 1uF 25V; footprint Capacitor_SMD:CP_Elec_10x10 -> Capacitor_SMD:C_0805_2012Metric
- C15, C28, C42: value 1uF 25V -> 470uF 25V; footprint Capacitor_SMD:C_0805_2012Metric -> Capacitor_SMD:CP_Elec_10x10
- C16: value DNP-1uF 25V -> 1uF 25V
- C19: value 100nf -> 470uF 25V; footprint Capacitor_SMD:C_0603_1608Metric -> Capacitor_SMD:CP_Elec_10x10
- C2: value 100nf -> DNP-1uF 25V; footprint Capacitor_SMD:C_0603_1608Metric -> Capacitor_SMD:C_0805_2012Metric
- C21: value 1uF 25V -> 10uF 25V; footprint Capacitor_SMD:C_0805_2012Metric -> Capacitor_SMD:C_1206_3216Metric
- C32, C88, C89, C90, C91: value 470uF 25V -> 100nf; footprint Capacitor_SMD:CP_Elec_10x10 -> Capacitor_SMD:C_0603_1608Metric
- C4: value DNP-1uF 25V -> 10uF 25V; footprint Capacitor_SMD:C_0805_2012Metric -> Capacitor_SMD:C_1206_3216Metric
- D14: value 40V 1A -> 5Vw; footprint Diode_SMD:D_SOD-123 -> Package_TO_SOT_SMD:SOT-23
- D16, D8: value 5Vw -> 40V 1A; footprint Package_TO_SOT_SMD:SOT-23 -> Diode_SMD:D_SOD-123
- D4, D9: value 5Vw -> 5Vw; footprint Diode_SMD:D_SMA -> Package_TO_SOT_SMD:SOT-23
- D5: value 12Vw -> 5Vw
- D6: value 40V 1A -> 12Vw; footprint Diode_SMD:D_SOD-123 -> Diode_SMD:D_SMA
- D7: value 5Vw -> 5Vw; footprint Package_TO_SOT_SMD:SOT-23 -> Diode_SMD:D_SMA
- J15: value Conn_01x02_Female -> SDS-50J; footprint Connector_JST:JST_XH_B2B-XH-A_1x02_P2.50mm_Vertical -> rainboard_fp:CUI_SDS-50J
- J17, J20, J21: value Conn_01x02_Female -> PH2-06-UA; footprint Connector_JST:JST_XH_B2B-XH-A_1x02_P2.50mm_Vertical -> Connector_PinHeader_2.54mm:PinHeader_2x03_P2.54mm_Vertical
- J18, J19: value Conn_01x02_Female -> Conn_01x03; footprint Connector_JST:JST_XH_B2B-XH-A_1x02_P2.50mm_Vertical -> Connector_JST:JST_XH_B3B-XH-AM_1x03_P2.50mm_Vertical
- J2: value USB_B -> SDS-50J; footprint rainboard_fp:UJ2-BH-1-TH -> rainboard_fp:CUI_SDS-50J
- J3: value Conn_01x03 -> USB_B; footprint Connector_JST:JST_XH_B3B-XH-AM_1x03_P2.50mm_Vertical -> rainboard_fp:UJ2-BH-1-TH
- J4: value Conn_01x03 -> Conn_01x02_Female; footprint Connector_JST:JST_XH_B3B-XH-AM_1x03_P2.50mm_Vertical -> Connector_JST:JST_XH_B2B-XH-A_1x02_P2.50mm_Vertical
- J5, J8, J9: value PH2-06-UA -> Conn_01x02_Female; footprint Connector_PinHeader_2.54mm:PinHeader_2x03_P2.54mm_Vertical -> Connector_JST:JST_XH_B2B-XH-A_1x02_P2.50mm_Vertical
- J6, J7: value SDS-50J -> Conn_01x02_Female; footprint rainboard_fp:CUI_SDS-50J -> Connector_JST:JST_XH_B2B-XH-A_1x02_P2.50mm_Vertical
- Q1: value DUAL 30V NMOS -> 30V 10mOhm; footprint Package_TO_SOT_SMD:SOT-363_SC-70-6 -> Package_SO:PowerPAK_SO-8_Single
- Q3: value 30V 10mOhm -> DUAL 30V NMOS; footprint Package_SO:PowerPAK_SO-8_Single -> Package_TO_SOT_SMD:SOT-363_SC-70-6
- R1: value 100k -> 210R; footprint Resistor_SMD:R_0603_1608Metric -> Resistor_SMD:R_0805_2012Metric
- R10, R12: value 100k -> 19.1k
- R11, R2: value 100k -> 11R
- R13: value 19.1k -> 100k
- R16: value 100k -> DNP-210R; footprint Resistor_SMD:R_0603_1608Metric -> Resistor_SMD:R_0805_2012Metric
- R17, R36, R7: value 11R -> 100k
- R18: value DNP-4.7k -> 4.7k
- R19, R35: value 4.7k -> 100k
- R20, R22, R29, R31, R39: value 11R -> 19.1k
- R21: value 19.1k -> 210R; footprint Resistor_SMD:R_0603_1608Metric -> Resistor_SMD:R_0805_2012Metric
- R23: value 210R -> 19.1k; footprint Resistor_SMD:R_0805_2012Metric -> Resistor_SMD:R_0603_1608Metric
- R25, R5: value 210R -> 11R; footprint Resistor_SMD:R_0805_2012Metric -> Resistor_SMD:R_0603_1608Metric
- R26: value DNP-210R -> 210R
- R27, R34, R44, R46: value 19.1k -> 4.7k
- R3, R4, R42, R51: value 4.7k -> 11R
- R30: value 210R -> 4.7k; footprint Resistor_SMD:R_0805_2012Metric -> Resistor_SMD:R_0603_1608Metric
- R32, R48: value 4.7k -> 19.1k
- R37, R38, R9: value 11R -> 4.7k
- R43, R47, R49, R53: value 19.1k -> 11R
- R45: value 4.7k -> DNP-4.7k
- R8: value 11R -> 210R; footprint Resistor_SMD:R_0603_1608Metric -> Resistor_SMD:R_0805_2012Metric
- SW10, SW11, SW12, SW13, SW14, SW15, SW16, SW5, SW52, SW6, SW7, SW8, SW9: footprint rainboard_newfighter:Sanwa-OBSF24-v2 -> rainboard_fp:Sanwa-OBSF24-v2
- U1: value RT8298 -> 6N137; footprint Package_SO:SOIC-8-1EP_3.9x4.9mm_P1.27mm_EP2.41x3.3mm_ThermalVias -> rainboard_fp:COUPL_6N138SDM
- U2: value ATmega16U2-MU -> RT8298; footprint Package_DFN_QFN:QFN-32-1EP_5x5mm_P0.5mm_EP3.1x3.1mm -> Package_SO:SOIC-8-1EP_3.9x4.9mm_P1.27mm_EP2.41x3.3mm_ThermalVias
- U3: value 6N137 -> 74HC14; footprint rainboard_fp:COUPL_6N138SDM -> Package_SO:TSSOP-14_4.4x5mm_P0.65mm
- U4: value 74HC14 -> ATmega16U2-MU; footprint Package_SO:TSSOP-14_4.4x5mm_P0.65mm -> Package_DFN_QFN:QFN-32-1EP_5x5mm_P0.5mm_EP3.1x3.1mm
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Connections:
- C1 pad 1: 12V_FILT -> Net-(C1-Pad1)
- C11 pad 1: Net-(C11-Pad1) -> 5V_MCU
- C12 pad 1: 12V_FILT -> Net-(C12-Pad1)
- C13 pad 1: 5V_USB -> 12V_FILT
- C14 pad 1: 12V_FILT -> 5V_USB
- C15 pad 1: Net-(C15-Pad1) -> 12V_FILT
- C15 pad 2: Net-(C15-Pad2) -> GND
- C16 pad 2: GND -> Net-(C16-Pad2)
- C18 pad 1: Net-(C18-Pad1) -> BARREL_DETECT
- C19 pad 1: BARREL_DETECT -> 5V_MCU
- C2 pad 1: AREF -> Net-(C2-Pad1)
- C2 pad 2: GNDA -> GND
- C20 pad 1: 5V_MCU -> 5V_POW
- C28 pad 1: 5V_MCU -> 5V_POW
- C29 pad 1: Net-(C29-Pad1) -> AREF
- C29 pad 2: GND -> GNDA
- C30 pad 1: 5V_POW -> MCU2_RST
- C31 pad 1: 5V_MCU -> Net-(C31-Pad1)
- C32 pad 1: 5V_POW -> MCU3_RST
- C33 pad 1: MCU3_RST -> 5V_USB
- C34 pad 1: 5V_MCU -> Net-(C34-Pad1)
- C34 pad 2: GND -> Net-(C34-Pad2)
- C35 pad 1: MCU2_RST -> 5V_USB
- C36 pad 1: Net-(C36-Pad1) -> 5V_MCU
- C37 pad 1: MCU1_RST -> 5V_MCU
- C38 pad 1: 5VA_MCU -> Net-(C38-Pad1)
- C39 pad 1: 5V_USB -> 5V_MCU
- C4 pad 1: Net-(C4-Pad1) -> 12V_FILT
- C40 pad 1: Net-(C40-Pad1) -> 5V_MCU
- C40 pad 2: Net-(C40-Pad2) -> GND
- C41 pad 1: 5V_USB -> 5VA_MCU
- C42 pad 1: 5V_MCU -> 5VA_MCU
- C43 pad 1: 5V_MCU -> 5V_USB
- C44 pad 1: Net-(C44-Pad1) -> 5V_USB
- C45 pad 1: 5V_MCU -> MCU1_RST
- C46 pad 1: 5V_MCU -> Net-(C46-Pad1)
- C47 pad 1: 5VA_MCU -> AREF
- C48 pad 1: 5V_USB -> 5V_MCU
- C49 pad 1: 5V_USB -> 5V_MCU
- C50 pad 1: AREF -> Net-(C50-Pad1)
- D10 pad 1: Net-(C15-Pad2) -> 5V_MCU
- D10 pad 2: GND -> Net-(D10-Pad2)
- D11 pad 2: Net-(D11-Pad2) -> 5V_USB
- D12 pad 1: 5V_MCU -> VLED
- D12 pad 2: 5V_USB -> /PCBMountButtons/FIRST_DIN
- D13 pad 3: Net-(D13-Pad3) -> GND
- D14 pad 1: VLED -> softpot-2
- D14 pad 2: /PCBMountButtons/FIRST_DIN -> softpot-1
- D15 pad 1: Net-(D15-Pad1) -> AREF
- D15 pad 2: Net-(D15-Pad2) -> BREF
- D16 pad 1: Net-(D16-Pad1) -> 5V_MCU
- D16 pad 2: Net-(D16-Pad2) -> MCU2_RST
- D17 pad 2: MCU2_RST -> MCU3_RST
- D3 pad 1: D- -> Net-(D3-Pad1)
- D3 pad 2: D+ -> Net-(D3-Pad2)
- D3 pad 3: GND -> Net-(D3-Pad3)
- D35 pad 4: /PCBMountButtons/FIRST_DIN -> /PCBMountButtons/sheet5FFC64B5/DIN
- D36 pad 4: /PCBMountButtons/sheet6019597E/DIN -> /PCBMountButtons/sheet5FFC64BB/DIN
- D37 pad 4: /PCBMountButtons/sheet61ABE4BE/DIN -> /PCBMountButtons/sheet5FFC64CF/DIN
- D38 pad 4: /PCBMountButtons/sheet61AC3886/DIN -> /PCBMountButtons/sheet5FFC64F0/DIN
- D39 pad 4: /PCBMountButtons/sheet61AC389A/DIN -> /PCBMountButtons/sheet5FFC64F7/DIN
- D4 pad 1: Net-(C11-Pad1) -> D-
- D4 pad 2: GND -> D+
- D40 pad 4: /PCBMountButtons/sheet61ACB861/DIN -> /PCBMountButtons/sheet5FFC6517/DIN
- D41 pad 4: /PCBMountButtons/sheet61ACB876/DIN -> /PCBMountButtons/sheet5FFC651D/DIN
- D42 pad 4: /PCBMountButtons/sheet61ACB899/DIN -> /PCBMountButtons/sheet5FFC6531/DIN
- D43 pad 4: /PCBMountButtons/sheet61AD1E3C/DIN -> /PCBMountButtons/sheet5FFD985B/DIN
- D44 pad 4: /PCBMountButtons/sheet61AD1E5E/DIN -> /PCBMountButtons/sheet5FFD9863/DIN
- D45 pad 4: /PCBMountButtons/sheet61AD1E64/DIN -> /PCBMountButtons/sheet5FFD9877/DIN
- D46 pad 4: /PCBMountButtons/sheet61AD1E79/DIN -> /PCBMountButtons/sheet5FFD988B/DIN
- D47 pad 4: /PCBMountButtons/sheet5FFC6464/DIN -> /PCBMountButtons/sheet5FFD98AC/DIN
- D48 pad 4: /PCBMountButtons/sheet5FFC646C/DIN -> /PCBMountButtons/sheet5FFD98B2/DIN
- D49 pad 4: /PCBMountButtons/sheet5FFC6480/DIN -> /PCBMountButtons/sheet5FFD98C6/DIN
- D5 pad 1: 12V_FILT -> Net-(C10-Pad1)
- D50 pad 4: /PCBMountButtons/sheet5FFC6494/DIN -> /PCBMountButtons/sheet5FFD98E7/DIN
- D51 pad 4: /PCBMountButtons/sheet5FFC64B5/DIN -> /PCBMountButtons/sheet5FFD98EE/DIN
- D52 pad 4: /PCBMountButtons/sheet5FFC64BB/DIN -> /PCBMountButtons/sheet5FFD990E/DIN
- D53 pad 4: /PCBMountButtons/sheet5FFC64CF/DIN -> /PCBMountButtons/sheet5FFD9914/DIN
- D54 pad 4: /PCBMountButtons/sheet5FFC64F0/DIN -> /PCBMountButtons/sheet5FFD9928/DIN
- D55 pad 4: /PCBMountButtons/sheet5FFC64F7/DIN -> /PCBMountButtons/sheet5FFFA930/DIN
- D56 pad 4: /PCBMountButtons/sheet5FFC6517/DIN -> /PCBMountButtons/sheet5FFFA938/DIN
- D57 pad 4: /PCBMountButtons/sheet5FFC651D/DIN -> /PCBMountButtons/sheet5FFFA94C/DIN
- D58 pad 4: /PCBMountButtons/sheet5FFC6531/DIN -> /PCBMountButtons/sheet5FFFA960/DIN
- D59 pad 4: /PCBMountButtons/sheet5FFD985B/DIN -> /PCBMountButtons/sheet5FFFA981/DIN
- D6 pad 1: 5V_MCU -> 12V_FILT
- D6 pad 2: MCU3_RST -> GND
- D60 pad 4: /PCBMountButtons/sheet5FFD9863/DIN -> /PCBMountButtons/sheet5FFFA987/DIN
- D61 pad 4: /PCBMountButtons/sheet5FFD9877/DIN -> /PCBMountButtons/sheet5FFFA99B/DIN
- D62 pad 4: /PCBMountButtons/sheet5FFD988B/DIN -> /PCBMountButtons/sheet5FFFA9BC/DIN
- D63 pad 4: /PCBMountButtons/sheet5FFD98AC/DIN -> /PCBMountButtons/sheet5FFFA9C3/DIN
- D64 pad 4: /PCBMountButtons/sheet5FFD98B2/DIN -> /PCBMountButtons/sheet5FFFA9E3/DIN
- D65 pad 4: /PCBMountButtons/sheet5FFD98C6/DIN -> /PCBMountButtons/sheet5FFFA9E9/DIN
- D66 pad 4: /PCBMountButtons/sheet5FFD98E7/DIN -> /PCBMountButtons/sheet5FFFA9FD/DIN
- D67 pad 4: /PCBMountButtons/sheet5FFD98EE/DIN -> /PCBMountButtons/sheet6001C156/DIN
- D68 pad 4: /PCBMountButtons/sheet5FFD990E/DIN -> /PCBMountButtons/sheet6001C15E/DIN
- D69 pad 4: /PCBMountButtons/sheet5FFD9914/DIN -> /PCBMountButtons/sheet6001C172/DIN
- D7 pad 1: softpot-2 -> 5V_USB
- D7 pad 2: softpot-1 -> GND
- D70 pad 4: /PCBMountButtons/sheet5FFD9928/DIN -> /PCBMountButtons/sheet6001C186/DIN
- D71 pad 4: /PCBMountButtons/sheet5FFFA930/DIN -> /PCBMountButtons/sheet6001C1A7/DIN
- D72 pad 4: /PCBMountButtons/sheet5FFFA938/DIN -> /PCBMountButtons/sheet6001C1AD/DIN
- D73 pad 4: /PCBMountButtons/sheet5FFFA94C/DIN -> /PCBMountButtons/sheet6001C1C1/DIN
- D74 pad 4: /PCBMountButtons/sheet5FFFA960/DIN -> /PCBMountButtons/sheet6001C1E2/DIN
- D75 pad 4: /PCBMountButtons/sheet5FFFA981/DIN -> /PCBMountButtons/sheet6001C1E9/DIN
- D76 pad 4: /PCBMountButtons/sheet5FFFA987/DIN -> /PCBMountButtons/sheet6112CF44/DIN
- D77 pad 4: /PCBMountButtons/sheet5FFFA99B/DIN -> /PCBMountButtons/sheet61155765/DIN
- D78 pad 4: /PCBMountButtons/sheet5FFFA9BC/DIN -> /PCBMountButtons/sheet611F5592/DIN
- D79 pad 4: /PCBMountButtons/sheet5FFFA9C3/DIN -> /PCBMountButtons/sheet6120995A/DIN
- D8 pad 1: AREF -> Net-(C16-Pad2)
- D8 pad 2: BREF -> GND
- D9 pad 1: 5V_USB -> Net-(D9-Pad1)
- D9 pad 2: GND -> Net-(D9-Pad2)
- F2 pad 1: Net-(C11-Pad1) -> Net-(C10-Pad1)
- J10 pad 1: BTNX-1 -> BTNX-4
- J11 pad 1: BTNX-2 -> BTNX-5
- J12 pad 1: BTNX-3 -> Net-(J12-Pad1)
- J13 pad 1: BTNX-7 -> Net-(J13-Pad1)
- J14 pad 1: BTNX-8 -> Net-(J14-Pad1)
- J15 pad 1: BTNX-9 -> Net-(J15-Pad1)
- J16 pad 1: BTNX-4 -> Net-(J16-Pad1)
- J17 pad 1: BTNX-5 -> MCU2_MISO2
- J17 pad 2: GND -> 5V_MCU
- J18 pad 1: BTNX-6 -> AREF
- J18 pad 2: GND -> softpot-1
- J19 pad 1: BTNX-10 -> AREF
- J19 pad 2: GND -> softpot-2
- J2 pad 1: Net-(F2-Pad2) -> Net-(J2-Pad1)
- J2 pad 2: Net-(J2-Pad2) -> Net-(C2-Pad1)
- J2 pad 4: GND -> Net-(J2-Pad4)
- J2 pad 5: Net-(FB1-Pad2) -> Net-(D3-Pad3)
- J20 pad 1: BTNX-11 -> MCU3_MISO3
- J20 pad 2: GND -> 5V_MCU
- J21 pad 1: BTNX-12 -> MCU1_MISO
- J21 pad 2: GND -> 5V_MCU
- J3 pad 1: AREF -> Net-(F2-Pad2)
- J3 pad 2: softpot-1 -> Net-(J3-Pad2)
- J3 pad 3: BREF -> Net-(J3-Pad3)
- J4 pad 1: AREF -> BTNX-1
- J4 pad 2: softpot-2 -> GND
- J5 pad 1: MCU3_MISO3 -> BTNX-2
- J5 pad 2: 5V_MCU -> GND
- J6 pad 1: Net-(J6-Pad1) -> BTNX-3
- J6 pad 2: Net-(C16-Pad1) -> GND
- J7 pad 1: Net-(J7-Pad1) -> BTNX-6
- J8 pad 1: MCU2_MISO2 -> BTNX-7
- J8 pad 2: 5V_MCU -> GND
- J9 pad 1: MCU1_MISO -> BTNX-8
- J9 pad 2: 5V_MCU -> GND
- JP1 pad 1: 5V_USB -> 5V_POW
- JP1 pad 2: Net-(JP1-Pad2) -> VLED
- JP2 pad 1: 5V_POW -> Net-(C34-Pad2)
- JP2 pad 2: VLED -> MCU1_RST
- JP3 pad 1: Net-(C40-Pad2) -> 5V_USB
- JP3 pad 2: MCU1_RST -> Net-(JP3-Pad2)
- L2 pad 2: Net-(C11-Pad1) -> Net-(C10-Pad1)
- L3 pad 2: Net-(C15-Pad2) -> Net-(C16-Pad2)
- L4 pad 1: Net-(D11-Pad2) -> Net-(D10-Pad2)
- Q1 pad 2: PROG_CTRL_1 -> GND
- Q1 pad 3: MCU2_MOSI2 -> GND
- Q1 pad 4: GND -> Net-(Q1-Pad4)
- Q1 pad 5: PROG_CTRL_2 -> Net-(C16-Pad2)
- Q2 pad 2: RST_2560 -> PROG_CTRL_1
- Q2 pad 3: Net-(Q2-Pad3) -> MCU2_MOSI2
- Q2 pad 4: Net-(Q2-Pad4) -> GND
- Q2 pad 5: Net-(Q2-Pad5) -> PROG_CTRL_2
- Q2 pad 6: MCU1_RST -> MCU2_RST
- Q3 pad 1: GND -> Net-(Q3-Pad1)
- Q3 pad 2: GND -> Net-(Q3-Pad2)
- Q3 pad 3: GND -> MCU1_RST
- Q3 pad 4: Net-(Q3-Pad4) -> GND
- Q3 pad 5: Net-(C15-Pad2) -> RST_2560
- R1 pad 1: softpot-1 -> Net-(J2-Pad4)
- R1 pad 2: GNDA -> Net-(D3-Pad1)
- R10 pad 1: Net-(R10-Pad1) -> BTN1a
- R10 pad 2: 12V_FILT -> Net-(J12-Pad1)
- R100 pad 1: /PCBMountButtons/sheet5FFFA987/DOUT -> /PCBMountButtons/sheet5FFFA9E3/DOUT
- R100 pad 2: /PCBMountButtons/sheet5FFFA99B/DIN -> /PCBMountButtons/sheet5FFFA9E9/DIN
- R101 pad 1: /PCBMountButtons/sheet5FFD98B2/DOUT -> /PCBMountButtons/sheet5FFD990E/DOUT
- R101 pad 2: /PCBMountButtons/sheet5FFD98C6/DIN -> /PCBMountButtons/sheet5FFD9914/DIN
- R102 pad 1: /PCBMountButtons/sheet5FFC64BB/DOUT -> /PCBMountButtons/sheet5FFC6517/DOUT
- R102 pad 2: /PCBMountButtons/sheet5FFC64CF/DIN -> /PCBMountButtons/sheet5FFC651D/DIN
- R103 pad 1: /PCBMountButtons/sheet61ACB861/DOUT -> /PCBMountButtons/sheet61AD1E5E/DOUT
- R103 pad 2: /PCBMountButtons/sheet61ACB876/DIN -> /PCBMountButtons/sheet61AD1E64/DIN
- R104 pad 1: /PCBMountButtons/sheet6001C1C1/DOUT -> /PCBMountButtons/sheet61155765/DOUT
- R104 pad 2: /PCBMountButtons/sheet6001C1E2/DIN -> /PCBMountButtons/sheet611F5592/DIN
- R105 pad 1: /PCBMountButtons/sheet5FFFA99B/DOUT -> /PCBMountButtons/sheet5FFFA9E9/DOUT
- R105 pad 2: /PCBMountButtons/sheet5FFFA9BC/DIN -> /PCBMountButtons/sheet5FFFA9FD/DIN
- R106 pad 1: /PCBMountButtons/sheet5FFD98C6/DOUT -> /PCBMountButtons/sheet5FFD9914/DOUT
- R106 pad 2: /PCBMountButtons/sheet5FFD98E7/DIN -> /PCBMountButtons/sheet5FFD9928/DIN
- R107 pad 1: /PCBMountButtons/sheet5FFC64CF/DOUT -> /PCBMountButtons/sheet5FFC651D/DOUT
- R107 pad 2: /PCBMountButtons/sheet5FFC64F0/DIN -> /PCBMountButtons/sheet5FFC6531/DIN
- R108 pad 1: /PCBMountButtons/sheet61ACB876/DOUT -> /PCBMountButtons/sheet61AD1E64/DOUT
- R108 pad 2: /PCBMountButtons/sheet61ACB899/DIN -> /PCBMountButtons/sheet61AD1E79/DIN
- R109 pad 1: /PCBMountButtons/sheet6001C1E2/DOUT -> /PCBMountButtons/sheet611F5592/DOUT
- R109 pad 2: /PCBMountButtons/sheet6001C1E9/DIN -> /PCBMountButtons/sheet6120995A/DIN
- R11 pad 1: BARREL_DETECT -> Net-(D9-Pad1)
- R11 pad 2: GND -> Net-(R11-Pad2)
- R110 pad 1: /PCBMountButtons/sheet5FFFA9BC/DOUT -> /PCBMountButtons/sheet5FFFA9FD/DOUT
- R110 pad 2: /PCBMountButtons/sheet5FFFA9C3/DIN -> /PCBMountButtons/sheet6001C156/DIN
- R111 pad 1: /PCBMountButtons/sheet5FFD98E7/DOUT -> /PCBMountButtons/sheet5FFD9928/DOUT
- R111 pad 2: /PCBMountButtons/sheet5FFD98EE/DIN -> /PCBMountButtons/sheet5FFFA930/DIN
- R112 pad 1: /PCBMountButtons/sheet5FFC64F0/DOUT -> /PCBMountButtons/sheet5FFC6531/DOUT
- R112 pad 2: /PCBMountButtons/sheet5FFC64F7/DIN -> /PCBMountButtons/sheet5FFD985B/DIN
- R113 pad 1: /PCBMountButtons/sheet61ACB899/DOUT -> /PCBMountButtons/sheet61AD1E79/DOUT
- R113 pad 2: /PCBMountButtons/sheet61AD1E3C/DIN -> /PCBMountButtons/sheet5FFC6464/DIN
- R114 pad 1: /PCBMountButtons/sheet6001C1E9/DOUT -> /PCBMountButtons/sheet6019597D/DOUT
- R114 pad 2: /PCBMountButtons/FINAL_DOUT -> Net-(D19-Pad2)
- R115 pad 1: /PCBMountButtons/sheet5FFFA9C3/DOUT -> /PCBMountButtons/sheet6019597E/DOUT
- R115 pad 2: /PCBMountButtons/sheet5FFFA9E3/DIN -> Net-(D20-Pad2)
- R116 pad 1: /PCBMountButtons/sheet5FFD98EE/DOUT -> /PCBMountButtons/sheet61ABE4BE/DOUT
- R116 pad 2: /PCBMountButtons/sheet5FFD990E/DIN -> Net-(D21-Pad2)
- R117 pad 1: /PCBMountButtons/sheet5FFC64F7/DOUT -> /PCBMountButtons/sheet61AC3886/DOUT
- R117 pad 2: /PCBMountButtons/sheet5FFC6517/DIN -> Net-(D22-Pad2)
- R118 pad 1: /PCBMountButtons/sheet61AD1E3C/DOUT -> /PCBMountButtons/sheet61AC389A/DOUT
- R118 pad 2: /PCBMountButtons/sheet61AD1E5E/DIN -> Net-(D23-Pad2)
- R119 pad 1: /PCBMountButtons/sheet5FFFA9E3/DOUT -> /PCBMountButtons/sheet61ACB861/DOUT
- R119 pad 2: /PCBMountButtons/sheet5FFFA9E9/DIN -> Net-(D24-Pad2)
- R12 pad 1: 5V_POW -> BTN1b
- R12 pad 2: Net-(R12-Pad2) -> Net-(J12-Pad1)
- R120 pad 1: /PCBMountButtons/sheet5FFD990E/DOUT -> /PCBMountButtons/sheet61ACB876/DOUT
- R120 pad 2: /PCBMountButtons/sheet5FFD9914/DIN -> Net-(D25-Pad2)
- R121 pad 1: /PCBMountButtons/sheet5FFC6517/DOUT -> /PCBMountButtons/sheet61ACB899/DOUT
- R121 pad 2: /PCBMountButtons/sheet5FFC651D/DIN -> Net-(D26-Pad2)
- R122 pad 1: /PCBMountButtons/sheet61AD1E5E/DOUT -> /PCBMountButtons/sheet61AD1E3C/DOUT
- R122 pad 2: /PCBMountButtons/sheet61AD1E64/DIN -> Net-(D27-Pad2)
- R123 pad 1: /PCBMountButtons/sheet5FFFA9E9/DOUT -> /PCBMountButtons/sheet61AD1E5E/DOUT
- R123 pad 2: /PCBMountButtons/sheet5FFFA9FD/DIN -> Net-(D28-Pad2)
- R124 pad 1: /PCBMountButtons/sheet5FFD9914/DOUT -> /PCBMountButtons/sheet61AD1E64/DOUT
- R124 pad 2: /PCBMountButtons/sheet5FFD9928/DIN -> Net-(D29-Pad2)
- R125 pad 1: /PCBMountButtons/sheet5FFC651D/DOUT -> /PCBMountButtons/sheet61AD1E79/DOUT
- R125 pad 2: /PCBMountButtons/sheet5FFC6531/DIN -> Net-(D30-Pad2)
- R126 pad 1: /PCBMountButtons/sheet61AD1E64/DOUT -> /PCBMountButtons/sheet5FFC6464/DOUT
- R126 pad 2: /PCBMountButtons/sheet61AD1E79/DIN -> Net-(D31-Pad2)
- R127 pad 1: /PCBMountButtons/sheet5FFFA9FD/DOUT -> /PCBMountButtons/sheet5FFC646C/DOUT
- R127 pad 2: /PCBMountButtons/sheet6001C156/DIN -> Net-(D32-Pad2)
- R128 pad 1: /PCBMountButtons/sheet5FFD9928/DOUT -> /PCBMountButtons/sheet5FFC6480/DOUT
- R128 pad 2: /PCBMountButtons/sheet5FFFA930/DIN -> Net-(D33-Pad2)
- R129 pad 1: /PCBMountButtons/sheet5FFC6531/DOUT -> /PCBMountButtons/sheet5FFC6494/DOUT
- R129 pad 2: /PCBMountButtons/sheet5FFD985B/DIN -> Net-(D34-Pad2)
- R13 pad 1: Net-(R12-Pad2) -> BARREL_DETECT
- R130 pad 1: /PCBMountButtons/sheet61AD1E79/DOUT -> /PCBMountButtons/sheet5FFC64B5/DOUT
- R130 pad 2: /PCBMountButtons/sheet5FFC6464/DIN -> Net-(D35-Pad2)
- R131 pad 1: /PCBMountButtons/sheet6019597D/DOUT -> /PCBMountButtons/sheet5FFC64BB/DOUT
- R131 pad 2: Net-(D35-Pad2) -> Net-(D36-Pad2)
- R132 pad 1: /PCBMountButtons/sheet6019597E/DOUT -> /PCBMountButtons/sheet5FFC64CF/DOUT
- R132 pad 2: Net-(D36-Pad2) -> Net-(D37-Pad2)
- R133 pad 1: /PCBMountButtons/sheet61ABE4BE/DOUT -> /PCBMountButtons/sheet5FFC64F0/DOUT
- R133 pad 2: Net-(D37-Pad2) -> Net-(D38-Pad2)
- R134 pad 1: /PCBMountButtons/sheet61AC3886/DOUT -> /PCBMountButtons/sheet5FFC64F7/DOUT
- R134 pad 2: Net-(D38-Pad2) -> Net-(D39-Pad2)
- R135 pad 1: /PCBMountButtons/sheet61AC389A/DOUT -> /PCBMountButtons/sheet5FFC6517/DOUT
- R135 pad 2: Net-(D39-Pad2) -> Net-(D40-Pad2)
- R136 pad 1: /PCBMountButtons/sheet61ACB861/DOUT -> /PCBMountButtons/sheet5FFC651D/DOUT
- R136 pad 2: Net-(D40-Pad2) -> Net-(D41-Pad2)
- R137 pad 1: /PCBMountButtons/sheet61ACB876/DOUT -> /PCBMountButtons/sheet5FFC6531/DOUT
- R137 pad 2: Net-(D41-Pad2) -> Net-(D42-Pad2)
- R138 pad 1: /PCBMountButtons/sheet61ACB899/DOUT -> /PCBMountButtons/sheet5FFD985B/DOUT
- R138 pad 2: Net-(D42-Pad2) -> Net-(D43-Pad2)
- R139 pad 1: /PCBMountButtons/sheet61AD1E3C/DOUT -> /PCBMountButtons/sheet5FFD9863/DOUT
- R139 pad 2: Net-(D43-Pad2) -> Net-(D44-Pad2)
- R140 pad 1: /PCBMountButtons/sheet61AD1E5E/DOUT -> /PCBMountButtons/sheet5FFD9877/DOUT
- R140 pad 2: Net-(D44-Pad2) -> Net-(D45-Pad2)
- R141 pad 1: /PCBMountButtons/sheet61AD1E64/DOUT -> /PCBMountButtons/sheet5FFD988B/DOUT
- R141 pad 2: Net-(D45-Pad2) -> Net-(D46-Pad2)
- R142 pad 1: /PCBMountButtons/sheet61AD1E79/DOUT -> /PCBMountButtons/sheet5FFD98AC/DOUT
- R142 pad 2: Net-(D46-Pad2) -> Net-(D47-Pad2)
- R143 pad 1: /PCBMountButtons/sheet5FFC6464/DOUT -> /PCBMountButtons/sheet5FFD98B2/DOUT
- R143 pad 2: Net-(D47-Pad2) -> Net-(D48-Pad2)
- R144 pad 1: /PCBMountButtons/sheet5FFC646C/DOUT -> /PCBMountButtons/sheet5FFD98C6/DOUT
- R144 pad 2: Net-(D48-Pad2) -> Net-(D49-Pad2)
- R145 pad 1: /PCBMountButtons/sheet5FFC6480/DOUT -> /PCBMountButtons/sheet5FFD98E7/DOUT
- R145 pad 2: Net-(D49-Pad2) -> Net-(D50-Pad2)
- R146 pad 1: /PCBMountButtons/sheet5FFC6494/DOUT -> /PCBMountButtons/sheet5FFD98EE/DOUT
- R146 pad 2: Net-(D50-Pad2) -> Net-(D51-Pad2)
- R147 pad 1: /PCBMountButtons/sheet5FFC64B5/DOUT -> /PCBMountButtons/sheet5FFD990E/DOUT
- R147 pad 2: Net-(D51-Pad2) -> Net-(D52-Pad2)
- R148 pad 1: /PCBMountButtons/sheet5FFC64BB/DOUT -> /PCBMountButtons/sheet5FFD9914/DOUT
- R148 pad 2: Net-(D52-Pad2) -> Net-(D53-Pad2)
- R149 pad 1: /PCBMountButtons/sheet5FFC64CF/DOUT -> /PCBMountButtons/sheet5FFD9928/DOUT
- R149 pad 2: Net-(D53-Pad2) -> Net-(D54-Pad2)
- R15 pad 1: Net-(J6-Pad4) -> MCU3_LED_CTRL
- R15 pad 2: Net-(D13-Pad1) -> /PCBMountButtons/FIRST_DIN
- R150 pad 1: /PCBMountButtons/sheet5FFC64F0/DOUT -> /PCBMountButtons/sheet5FFFA930/DOUT
- R150 pad 2: Net-(D54-Pad2) -> Net-(D55-Pad2)
- R151 pad 1: /PCBMountButtons/sheet5FFC64F7/DOUT -> /PCBMountButtons/sheet5FFFA938/DOUT
- R151 pad 2: Net-(D55-Pad2) -> Net-(D56-Pad2)
- R152 pad 1: /PCBMountButtons/sheet5FFC6517/DOUT -> /PCBMountButtons/sheet5FFFA94C/DOUT
- R152 pad 2: Net-(D56-Pad2) -> Net-(D57-Pad2)
- R153 pad 1: /PCBMountButtons/sheet5FFC651D/DOUT -> /PCBMountButtons/sheet5FFFA960/DOUT
- R153 pad 2: Net-(D57-Pad2) -> Net-(D58-Pad2)
- R154 pad 1: /PCBMountButtons/sheet5FFC6531/DOUT -> /PCBMountButtons/sheet5FFFA981/DOUT
- R154 pad 2: Net-(D58-Pad2) -> Net-(D59-Pad2)
- R155 pad 1: /PCBMountButtons/sheet5FFD985B/DOUT -> /PCBMountButtons/sheet5FFFA987/DOUT
- R155 pad 2: Net-(D59-Pad2) -> Net-(D60-Pad2)
- R156 pad 1: /PCBMountButtons/sheet5FFD9863/DOUT -> /PCBMountButtons/sheet5FFFA99B/DOUT
- R156 pad 2: Net-(D60-Pad2) -> Net-(D61-Pad2)
- R157 pad 1: /PCBMountButtons/sheet5FFD9877/DOUT -> /PCBMountButtons/sheet5FFFA9BC/DOUT
- R157 pad 2: Net-(D61-Pad2) -> Net-(D62-Pad2)
- R158 pad 1: /PCBMountButtons/sheet5FFD988B/DOUT -> /PCBMountButtons/sheet5FFFA9C3/DOUT
- R158 pad 2: Net-(D62-Pad2) -> Net-(D63-Pad2)
- R159 pad 1: /PCBMountButtons/sheet5FFD98AC/DOUT -> /PCBMountButtons/sheet5FFFA9E3/DOUT
- R159 pad 2: Net-(D63-Pad2) -> Net-(D64-Pad2)
- R16 pad 1: BARREL_DETECT -> MCU2_LED_CTRL
- R16 pad 2: GND -> /PCBMountButtons/FIRST_DIN
- R160 pad 1: /PCBMountButtons/sheet5FFD98B2/DOUT -> /PCBMountButtons/sheet5FFFA9E9/DOUT
- R160 pad 2: Net-(D64-Pad2) -> Net-(D65-Pad2)
- R161 pad 1: /PCBMountButtons/sheet5FFD98C6/DOUT -> /PCBMountButtons/sheet5FFFA9FD/DOUT
- R161 pad 2: Net-(D65-Pad2) -> Net-(D66-Pad2)
- R162 pad 1: /PCBMountButtons/sheet5FFD98E7/DOUT -> /PCBMountButtons/sheet6001C156/DOUT
- R162 pad 2: Net-(D66-Pad2) -> Net-(D67-Pad2)
- R163 pad 1: /PCBMountButtons/sheet5FFD98EE/DOUT -> /PCBMountButtons/sheet6001C15E/DOUT
- R163 pad 2: Net-(D67-Pad2) -> Net-(D68-Pad2)
- R164 pad 1: /PCBMountButtons/sheet5FFD990E/DOUT -> /PCBMountButtons/sheet6001C172/DOUT
- R164 pad 2: Net-(D68-Pad2) -> Net-(D69-Pad2)
- R165 pad 1: /PCBMountButtons/sheet5FFD9914/DOUT -> /PCBMountButtons/sheet6001C186/DOUT
- R165 pad 2: Net-(D69-Pad2) -> Net-(D70-Pad2)
- R166 pad 1: /PCBMountButtons/sheet5FFD9928/DOUT -> /PCBMountButtons/sheet6001C1A7/DOUT
- R166 pad 2: Net-(D70-Pad2) -> Net-(D71-Pad2)
- R167 pad 1: /PCBMountButtons/sheet5FFFA930/DOUT -> /PCBMountButtons/sheet6001C1AD/DOUT
- R167 pad 2: Net-(D71-Pad2) -> Net-(D72-Pad2)
- R168 pad 1: /PCBMountButtons/sheet5FFFA938/DOUT -> /PCBMountButtons/sheet6001C1C1/DOUT
- R168 pad 2: Net-(D72-Pad2) -> Net-(D73-Pad2)
- R169 pad 1: /PCBMountButtons/sheet5FFFA94C/DOUT -> /PCBMountButtons/sheet6001C1E2/DOUT
- R169 pad 2: Net-(D73-Pad2) -> Net-(D74-Pad2)
- R17 pad 1: Net-(D13-Pad2) -> BARREL_DETECT
- R17 pad 2: Net-(D13-Pad1) -> GND
- R170 pad 1: /PCBMountButtons/sheet5FFFA960/DOUT -> /PCBMountButtons/sheet6001C1E9/DOUT
- R170 pad 2: Net-(D74-Pad2) -> Net-(D75-Pad2)
- R171 pad 1: /PCBMountButtons/sheet5FFFA981/DOUT -> /PCBMountButtons/sheet6112CF44/DOUT
- R171 pad 2: Net-(D75-Pad2) -> Net-(D76-Pad2)
- R172 pad 1: /PCBMountButtons/sheet5FFFA987/DOUT -> /PCBMountButtons/sheet61155765/DOUT
- R172 pad 2: Net-(D76-Pad2) -> Net-(D77-Pad2)
- R173 pad 1: /PCBMountButtons/sheet5FFFA99B/DOUT -> /PCBMountButtons/sheet611F5592/DOUT
- R173 pad 2: Net-(D77-Pad2) -> Net-(D78-Pad2)
- R174 pad 1: /PCBMountButtons/sheet5FFFA9BC/DOUT -> /PCBMountButtons/sheet6120995A/DOUT
- R174 pad 2: Net-(D78-Pad2) -> Net-(D79-Pad2)
- R18 pad 1: Net-(R18-Pad1) -> 5V_MCU
- R18 pad 2: GND -> Net-(J13-Pad1)
- R19 pad 1: 5V_MCU -> 5V_POW
- R19 pad 2: Net-(R18-Pad1) -> Net-(R19-Pad2)
- R2 pad 1: softpot-2 -> Net-(D2-Pad2)
- R2 pad 2: GNDA -> Net-(J3-Pad3)
- R20 pad 1: MCU3_LED_CTRL -> Net-(R19-Pad2)
- R20 pad 2: MCU3_MOSI3 -> GND
- R21 pad 1: 5V_MCU -> Net-(D9-Pad1)
- R21 pad 2: MCU2_RST -> Net-(D9-Pad2)
- R22 pad 1: MCU3_LED_CTRL -> /PCBMountButtons/FIRST_DIN
- R22 pad 2: Net-(R22-Pad2) -> GND
- R23 pad 1: Net-(R23-Pad1) -> BTN2a
- R23 pad 2: 5V_MCU -> Net-(J13-Pad1)
- R24 pad 1: BARREL_DETECT -> BTN2b
- R24 pad 2: Net-(C29-Pad1) -> Net-(J13-Pad1)
- R25 pad 1: MCU3_LED_CTRL -> 5V_MCU
- R25 pad 2: /PCBMountButtons/FIRST_DIN -> Net-(D13-Pad2)
- R26 pad 1: MCU2_LED_CTRL -> Net-(D13-Pad2)
- R26 pad 2: /PCBMountButtons/FIRST_DIN -> Net-(D13-Pad1)
- R27 pad 1: /PCBMountButtons/FIRST_DIN -> 5V_MCU
- R27 pad 2: GND -> Net-(J14-Pad1)
- R28 pad 1: 5V_MCU -> BTN3a
- R28 pad 2: MCU3_RST -> Net-(J14-Pad1)
- R29 pad 1: Net-(D15-Pad1) -> BTN3b
- R29 pad 2: Net-(R29-Pad2) -> Net-(J14-Pad1)
- R3 pad 1: 5VA_MCU -> Net-(D2-Pad1)
- R3 pad 2: AREF -> Net-(J3-Pad2)
- R30 pad 1: Net-(D15-Pad1) -> 5V_MCU
- R30 pad 2: Net-(D15-Pad2) -> Net-(J16-Pad1)
- R31 pad 1: 5V_MCU -> BTN4a
- R31 pad 2: Net-(D16-Pad2) -> Net-(J16-Pad1)
- R32 pad 1: PROG_CTRL_1 -> BTN4b
- R32 pad 2: GND -> Net-(J16-Pad1)
- R33 pad 1: PROG_CTRL_2 -> PROG_CTRL_1
- R34 pad 1: MCU1_RST -> PROG_CTRL_2
- R34 pad 2: 5V_MCU -> GND
- R35 pad 1: Net-(C40-Pad1) -> softpot-1
- R35 pad 2: GND -> GNDA
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
Commit message: position midi DIN, USB, and power barrel
Parts:
- moved J15 265.4 mm to (-41.9, 129.5)
- moved J3 261.7 mm to (0.00, 129.5)
- moved J1 220.7 mm to (42.0, 130.0), turned to 90 degrees
- moved J2 3.01 mm to (171.8, -49.8)

Commit message: position J4 through J16
Parts:
- moved J12 381.0 mm to (-144.3, 19.1)
- moved J13 341.1 mm to (-118.7, 54.7)
- moved J14 306.8 mm to (-99.2, 86.8)
- moved J16 298.4 mm to (-81.7, 119.9)
- moved J6 273.6 mm to (-18.7, -127.1)
- moved J7 272.9 mm to (-48.1, -127.1)
- moved J19 233.8 mm to (70.9, 120.0)
- moved J18 231.4 mm to (61.3, 132.8)
- moved J5 226.8 mm to (16.4, -124.8)
- moved J4 215.4 mm to (45.1, -126.9)
- moved J11 188.7 mm to (85.7, 100.1)
- moved J8 147.0 mm to (125.9, 22.2)
- moved J9 141.3 mm to (112.7, 50.9)
- moved J10 136.2 mm to (97.4, 76.8)
Changed lines of the file:
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@@
   )
   (module Connector_JST:JST_XH_B3B-XH-AM_1x03_P2.50mm_Vertical (layer F.Cu)
-    (at 233.57 -48)
+    (at 70.9295 119.9515)
     (descr "JST XH series connector, B3B-XH-AM, with boss (http://www.jst-mfg.com/product/pdf/eng/eXH.pdf), generated with kicad-footprint-generator")
     (tags "connector JST XH vertical boss")
@@
   )
   (module Connector_JST:JST_XH_B3B-XH-AM_1x03_P2.50mm_Vertical (layer F.Cu)
-    (at 219.49 -36.15)
+    (at 61.3175 132.7785)
     (descr "JST XH series connector, B3B-XH-AM, with boss (http://www.jst-mfg.com/product/pdf/eng/eXH.pdf), generated with kicad-footprint-generator")
     (tags "connector JST XH vertical boss")
@@
   )
   (module Connector_JST:JST_XH_B2B-XH-A_1x02_P2.50mm_Vertical (layer F.Cu)
-    (at 195.66 9.98)
+    (at -81.7245 119.888)
     (descr "JST XH series connector, B2B-XH-A (http://www.jst-mfg.com/product/pdf/eng/eXH.pdf), generated with kicad-footprint-generator")
     (tags "connector JST XH vertical")
@@
   )
   (module Connector_JST:JST_XH_B2B-XH-A_1x02_P2.50mm_Vertical (layer F.Cu)
-    (at 195.66 2.18)
+    (at -99.187 86.8045)
     (descr "JST XH series connector, B2B-XH-A (http://www.jst-mfg.com/product/pdf/eng/eXH.pdf), generated with kicad-footprint-generator")
     (tags "connector JST XH vertical")
@@
   )
   (module Connector_JST:JST_XH_B2B-XH-A_1x02_P2.50mm_Vertical (layer F.Cu)
-    (at 216.29 -9.8)
+    (at -118.6815 54.737)
     (descr "JST XH series connector, B2B-XH-A (http://www.jst-mfg.com/product/pdf/eng/eXH.pdf), generated with kicad-footprint-generator")
     (tags "connector JST XH vertical")
@@
   )
   (module Connector_JST:JST_XH_B2B-XH-A_1x02_P2.50mm_Vertical (layer F.Cu)
-    (at 233.38 -30.5)
+    (at -144.3355 19.1135)
     (descr "JST XH series connector, B2B-XH-A (http://www.jst-mfg.com/product/pdf/eng/eXH.pdf), generated with kicad-footprint-generator")
     (tags "connector JST XH vertical")
@@
   )
   (module Connector_JST:JST_XH_B2B-XH-A_1x02_P2.50mm_Vertical (layer F.Cu)
-    (at 223.93 -28.35)
+    (at 85.725 100.076)
     (descr "JST XH series connector, B2B-XH-A (http://www.jst-mfg.com/product/pdf/eng/eXH.pdf), generated with kicad-footprint-generator")
     (tags "connector JST XH vertical")
@@
   )
   (module Connector_JST:JST_XH_B2B-XH-A_1x02_P2.50mm_Vertical (layer F.Cu)
-    (at 205.8 -5.62)
+    (at 97.3855 76.835)
     (descr "JST XH series connector, B2B-XH-A (http://www.jst-mfg.com/product/pdf/eng/eXH.pdf), generated with kicad-footprint-generator")
     (tags "connector JST XH vertical")
@@
   )
   (module Connector_JST:JST_XH_B2B-XH-A_1x02_P2.50mm_Vertical (layer F.Cu)
-    (at 233.38 -22.7)
+    (at 112.7125 50.8635)
     (descr "JST XH series connector, B2B-XH-A (http://www.jst-mfg.com/product/pdf/eng/eXH.pdf), generated with kicad-footprint-generator")
     (tags "connector JST XH vertical")
@@
   )
   (module Connector_JST:JST_XH_B2B-XH-A_1x02_P2.50mm_Vertical (layer F.Cu)
-    (at 254.97 -48)
+    (at 125.857 22.225)
     (descr "JST XH series connector, B2B-XH-A (http://www.jst-mfg.com/product/pdf/eng/eXH.pdf), generated with kicad-footprint-generator")
     (tags "connector JST XH vertical")
@@
   )
   (module Connector_JST:JST_XH_B2B-XH-A_1x02_P2.50mm_Vertical (layer F.Cu)
-    (at 196.35 -5.62)
+    (at -48.0695 -127.0635)
     (descr "JST XH series connector, B2B-XH-A (http://www.jst-mfg.com/product/pdf/eng/eXH.pdf), generated with kicad-footprint-generator")
     (tags "connector JST XH vertical")
@@
   )
   (module Connector_JST:JST_XH_B2B-XH-A_1x02_P2.50mm_Vertical (layer F.Cu)
-    (at 240.77 -40.2)
+    (at -18.669 -127.0635)
     (descr "JST XH series connector, B2B-XH-A (http://www.jst-mfg.com/product/pdf/eng/eXH.pdf), generated with kicad-footprint-generator")
     (tags "connector JST XH vertical")
@@
   )
   (module Connector_JST:JST_XH_B2B-XH-A_1x02_P2.50mm_Vertical (layer F.Cu)
-    (at 216.29 -17.6)
+    (at 16.4465 -124.7775)
     (descr "JST XH series connector, B2B-XH-A (http://www.jst-mfg.com/product/pdf/eng/eXH.pdf), generated with kicad-footprint-generator")
     (tags "connector JST XH vertical")
@@
   )
   (module Connector_JST:JST_XH_B2B-XH-A_1x02_P2.50mm_Vertical (layer F.Cu)
-    (at 245.52 -48)
-    (descr "JST XH series connector, B2B-XH-A (http://www.jst-mfg.com/product/pdf/eng/eXH.pdf), generated with kicad-footprint-generator")
-    (tags "connector JST XH vertical")
+    (at 45.085 -126.873)
+    (descr "JST XH series connector, B2B-XH-A (http://www.jst-mfg.com/product/pdf/eng/eXH.pdf), generated with kicad-footprint-generator")
+    (tags "connector JST XH vertical")

Commit message: Footprints fixed, button orgin moved to allow placement of LEDs
Parts:
- J1: footprint Connector_BarrelJack:BarrelJack_Horizontal -> rainboard_fp:BarrelJack_Horizontal
- Q1: footprint Package_SO:PowerPAK_SO-8_Single -> rainboard_fp:PowerPAK_SO-8_Single
- U2: footprint Package_SO:SOIC-8-1EP_3.9x4.9mm_P1.27mm_EP2.41x3.3mm_ThermalVias -> rainboard_fp:SOIC-8-1EP_3.9x4.9mm_P1.27mm_EP2.41x3.3mm_ThermalVias
- U4: footprint Package_DFN_QFN:QFN-32-1EP_5x5mm_P0.5mm_EP3.1x3.1mm -> rainboard_fp:QFN33P50_500X500X60L40X24T300N
- moved J4 7.62 mm to (45.1, -119.3)
- moved J5 7.62 mm to (16.4, -117.2)
- moved J6 7.62 mm to (-18.7, -119.4)
- moved J7 7.62 mm to (-48.1, -119.4)
- moved SW1 7.62 mm to (-59.0, -94.6)
- moved SW10 7.62 mm to (44.2, -69.0)
- moved SW11 7.62 mm to (73.7, -69.0)
- moved SW12 7.62 mm to (-88.5, -43.5)
- moved SW13 7.62 mm to (-59.0, -43.5)
- moved SW14 7.62 mm to (-29.5, -43.5)
- moved SW15 7.62 mm to (0.00, -43.5)
- moved SW16 7.62 mm to (29.5, -43.5)
- moved SW17 7.62 mm to (59.0, -43.5)
- moved SW18 7.62 mm to (88.5, -43.5)
- moved SW2 7.62 mm to (-29.5, -94.6)
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