File: rainboard-pcb/kicad_proj/rainboard_newfighter/rainboard_newfighter.kicad_pcb (KiCad board)
At the start: 2 copper layers, 260 x 253.6 mm, 489 parts, among them J1 54-00167, J10 Conn_01x02_Female, J11 Conn_01x02_Female, J12 Conn_01x02_Female, J13 Conn_01x02_Female, J14 Conn_01x02_Female, J15 SDS-50J, J16 Conn_01x02_Female, J17 PH2-06-UA, J18 Conn_01x03, J19 Conn_01x03, J2 SDS-50J, J20 PH2-06-UA, J21 PH2-06-UA, J3 USB_B, J4 Conn_01x02_Female, J5 Conn_01x02_Female, J6 Conn_01x02_Female, J7 Conn_01x02_Female, J8 Conn_01x02_Female, J9 Conn_01x02_Female, Q2 DUAL 30V NMOS, Q3 DUAL 30V NMOS, SW1 SANWA-OBSF24, SW10 SANWA-OBSF24, SW11 SANWA-OBSF24, SW12 SANWA-OBSF24, SW13 SANWA-OBSF24, SW14 SANWA-OBSF24, SW15 SANWA-OBSF24, SW16 SANWA-OBSF24, SW17 SANWA-OBSF24, SW18 SANWA-OBSF24, SW19 SANWA-OBSF24, SW2 SANWA-OBSF24, SW20 SANWA-OBSF24, SW21 SANWA-OBSF24, SW22 SANWA-OBSF24, SW23 SANWA-OBSF24, SW24 SANWA-OBSF24, SW25 SANWA-OBSF24, SW26 SANWA-OBSF24, SW27 SANWA-OBSF24, SW28 SANWA-OBSF24, SW29 SANWA-OBSF24, SW3 SANWA-OBSF24, SW30 SANWA-OBSF24, SW31 SANWA-OBSF24, SW32 SANWA-OBSF24, SW33 SANWA-OBSF24, SW34 SANWA-OBSF24, SW35 SANWA-OBSF24, SW36 SANWA-OBSF24, SW37 SANWA-OBSF24, SW38 SANWA-OBSF24, SW39 SANWA-OBSF24, SW4 SANWA-OBSF24, SW40 SANWA-OBSF24, SW41 SANWA-OBSF24, SW42 SANWA-OBSF24, SW43 SANWA-OBSF24, SW44 SANWA-OBSF24, SW45 SANWA-OBSF24, SW46 SANWA-OBSF24, SW47 SANWA-OBSF24, SW48 SANWA-OBSF24, SW49 SANWA-OBSF24, SW5 SANWA-OBSF24, SW50 SANWA-OBSF24, SW51 SANWA-OBSF24, SW52 SANWA-OBSF24, SW53 SANWA-OBSF24, SW54 SANWA-OBSF24, SW55 SANWA-OBSF24, SW56 SANWA-OBSF24, SW57 SANWA-OBSF24, SW58 SANWA-OBSF24, SW59 SANWA-OBSF24, SW6 SANWA-OBSF24, SW60 SANWA-OBSF24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

Commit message: Starts PCB setup
Parts:
- U6: moved to B.Cu
- moved R9 398.0 mm to (-143.7, 27.7)
- moved R23 376.8 mm to (-119.0, 63.8)
- moved R12 366.9 mm to (-143.8, 24.4)
- moved R10 362.8 mm to (-143.8, 26.0)
- moved R30 357.3 mm to (-80.0, 125.1)
- moved R28 356.1 mm to (-98.1, 92.4)
- moved R24 351.6 mm to (-119.0, 59.7)
- moved R31 344.4 mm to (-80.1, 127.2)
- moved R174 343.1 mm to (146.6, 251.0)
- moved R29 343.0 mm to (-98.0, 94.4)
- moved C65 340.8 mm to (-57.3, -89.9), turned to 180 degrees
- moved R114 337.9 mm to (-53.4, -95.3), turned to 180 degrees
- moved R18 337.9 mm to (-119.0, 61.7)
- moved D19 337.2 mm to (-59.0, -93.7), turned to 180 degrees
- moved C66 336.6 mm to (-27.8, -89.9), turned to 180 degrees
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
Commit message: general placement of leds
Parts:
- C100, C101, C102, C103, C104, C105, C106, C107, C108, C109, C110, C111, C112, C113, C114, C115, C116, C117, C118, C119, C120, C121, C122, C123, C124, C125, C65, C66, C67, C68, C69, C70, C71, C72, C73, C74, C75, C76, C77, C78, C79, C80, C81, C82, C83, C84, C85, C86, C87, C88, C89, C90, C91, C92, C93, C94, C95, C96, C97, C98, C99, R100, R101, R102, R103, R104, R105, R106, R107, R108, R109, R110, R111, R112, R113, R114, R115, R116, R117, R118, R119, R120, R121, R122, R123, R124, R125, R126, R127, R128, R129, R130, R131, R132, R133, R134, R135, R136, R137, R138, R139, R140, R141, R142, R143, R144, R145, R146, R147, R148, R149, R150, R151, R152, R153, R154, R155, R156, R157, R158, R159, R160, R161, R162, R163, R164, R165, R166, R167, R168, R169, R170, R171, R172, R173, R174, R54, R55, R56, R57, R58, R59, R60, R61, R62, R63, R64, R65, R66, R67, R68, R69, R70, R71, R72, R73, R74, R75, R76, R77, R78, R79, R80, R81, R82, R83, R84, R85, R86, R87, R88, R89, R90, R91, R92, R93, R94, R95, R96, R97, R98, R99: moved to B.Cu
- moved C76 337.3 mm to (-88.5, -43.5), turned to 180 degrees
- moved R124 335.1 mm to (-79.5, -67.4)
- moved C75 333.6 mm to (-73.7, -69.0)
- moved R108 332.8 mm to (-94.2, -41.9)
- moved R125 332.3 mm to (-82.8, -45.1), turned to 180 degrees
- moved C91 332.3 mm to (-118.0, 7.62), turned to 180 degrees
- moved D30 331.8 mm to (-88.5, -43.5), turned to 180 degrees
- moved R139 328.6 mm to (-109.0, -16.3)
- moved D29 328.3 mm to (-73.7, -69.0)
- moved C90 327.6 mm to (-103.2, -17.9)
- moved D45 326.5 mm to (-118.0, 7.62), turned to 180 degrees
- moved R140 325.0 mm to (-112.3, 6.01), turned to 180 degrees
- moved R61 324.7 mm to (-119.8, 10.1), turned to 180 degrees
- moved C77 323.4 mm to (-59.0, -43.5), turned to 180 degrees
- moved C120 322.6 mm to (-73.7, 84.3)
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Routing:
- net GND: track 0.00 -> 241.7 mm, vias 0 -> 61
- net VLED: track 0.00 -> 240.5 mm, vias 0 -> 61
- net /PCBMountButtons/sheet6001C186/DOUT: track 0.00 -> 17.6 mm
- net /PCBMountButtons/sheet5FFC64CF/DOUT: track 0.00 -> 17.6 mm
- net /PCBMountButtons/sheet61AD1E79/DOUT: track 0.00 -> 17.6 mm
- net /PCBMountButtons/sheet5FFC64F0/DOUT: track 0.00 -> 17.6 mm
- net /PCBMountButtons/sheet5FFC6494/DOUT: track 0.00 -> 17.6 mm
- net /PCBMountButtons/sheet6001C1C1/DOUT: track 0.00 -> 17.6 mm
- net /PCBMountButtons/sheet6001C1A7/DOUT: track 0.00 -> 17.6 mm
- net /PCBMountButtons/sheet5FFFA9C3/DOUT: track 0.00 -> 17.6 mm
- net /PCBMountButtons/sheet5FFC64B5/DOUT: track 0.00 -> 17.6 mm
- net /PCBMountButtons/sheet6001C1E9/DOUT: track 0.00 -> 17.6 mm
- net /PCBMountButtons/sheet6001C1AD/DOUT: track 0.00 -> 17.6 mm
- net /PCBMountButtons/sheet5FFFA987/DOUT: track 0.00 -> 17.6 mm
- net /PCBMountButtons/sheet5FFFA9BC/DOUT: track 0.00 -> 17.6 mm
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
Commit message: prelim place & route
deleted extra R's layout & sch
Parts:
- removed R100, R101, R102, R103, R104, R105, R107, R109, R110, R111, R112, R113, R54, R55, R56, R57, R58, R60, R62, R63, R64, R65, R66, R67, R68, R69, R70, R71, R72, R73, R74, R75, R76, R77, R78, R79, R80, R81, R83, R84, R86, R87, R88, R90, R91, R92, R93, R94, R95, R96, R97, R98, R99: 210R, Resistor_SMD:R_0805_2012Metric
- moved J5 19.9 mm to (13.5, -103.7)
- moved J4 17.9 mm to (43.0, -103.5)
- moved J6 17.7 mm to (-16.0, -103.6)
- moved J7 17.6 mm to (-45.6, -103.6)
Connections:
- R114 pad 1: /PCBMountButtons/sheet6019597D/DOUT -> /PCBMountButtons/sheet6019597E/DIN
- R115 pad 1: /PCBMountButtons/sheet6019597E/DOUT -> /PCBMountButtons/sheet61ABE4BE/DIN
- R116 pad 1: /PCBMountButtons/sheet61ABE4BE/DOUT -> /PCBMountButtons/sheet61AC3886/DIN
- R117 pad 1: /PCBMountButtons/sheet61AC3886/DOUT -> /PCBMountButtons/sheet61AC389A/DIN
- R118 pad 1: /PCBMountButtons/sheet61AC389A/DOUT -> /PCBMountButtons/sheet61ACB861/DIN
- R119 pad 1: /PCBMountButtons/sheet61ACB861/DOUT -> /PCBMountButtons/sheet61ACB876/DIN
- R120 pad 1: /PCBMountButtons/sheet61ACB876/DOUT -> /PCBMountButtons/sheet61ACB899/DIN
- R121 pad 1: /PCBMountButtons/sheet61ACB899/DOUT -> /PCBMountButtons/sheet61AD1E3C/DIN
- R122 pad 1: /PCBMountButtons/sheet61AD1E3C/DOUT -> /PCBMountButtons/sheet61AD1E5E/DIN
- R123 pad 1: /PCBMountButtons/sheet61AD1E5E/DOUT -> /PCBMountButtons/sheet61AD1E64/DIN
- R124 pad 1: /PCBMountButtons/sheet61AD1E64/DOUT -> /PCBMountButtons/sheet61AD1E79/DIN
- R125 pad 1: /PCBMountButtons/sheet61AD1E79/DOUT -> /PCBMountButtons/sheet5FFC6464/DIN
- R126 pad 1: /PCBMountButtons/sheet5FFC6464/DOUT -> /PCBMountButtons/sheet5FFC646C/DIN
- R127 pad 1: /PCBMountButtons/sheet5FFC646C/DOUT -> /PCBMountButtons/sheet5FFC6480/DIN
- R128 pad 1: /PCBMountButtons/sheet5FFC6480/DOUT -> /PCBMountButtons/sheet5FFC6494/DIN
- R129 pad 1: /PCBMountButtons/sheet5FFC6494/DOUT -> /PCBMountButtons/sheet5FFC64B5/DIN
- R130 pad 1: /PCBMountButtons/sheet5FFC64B5/DOUT -> /PCBMountButtons/sheet5FFC64BB/DIN
- R131 pad 1: /PCBMountButtons/sheet5FFC64BB/DOUT -> /PCBMountButtons/sheet5FFC64CF/DIN
- R132 pad 1: /PCBMountButtons/sheet5FFC64CF/DOUT -> /PCBMountButtons/sheet5FFC64F0/DIN
- R133 pad 1: /PCBMountButtons/sheet5FFC64F0/DOUT -> /PCBMountButtons/sheet5FFC64F7/DIN
- R134 pad 1: /PCBMountButtons/sheet5FFC64F7/DOUT -> /PCBMountButtons/sheet5FFC6517/DIN
- R135 pad 1: /PCBMountButtons/sheet5FFC6517/DOUT -> /PCBMountButtons/sheet5FFC651D/DIN
- R136 pad 1: /PCBMountButtons/sheet5FFC651D/DOUT -> /PCBMountButtons/sheet5FFC6531/DIN
- R137 pad 1: /PCBMountButtons/sheet5FFC6531/DOUT -> /PCBMountButtons/sheet5FFD985B/DIN
- R138 pad 1: /PCBMountButtons/sheet5FFD985B/DOUT -> /PCBMountButtons/sheet5FFD9863/DIN
- R139 pad 1: /PCBMountButtons/sheet5FFD9863/DOUT -> /PCBMountButtons/sheet5FFD9877/DIN
- R140 pad 1: /PCBMountButtons/sheet5FFD9877/DOUT -> /PCBMountButtons/sheet5FFD988B/DIN
- R141 pad 1: /PCBMountButtons/sheet5FFD988B/DOUT -> /PCBMountButtons/sheet5FFD98AC/DIN
- R142 pad 1: /PCBMountButtons/sheet5FFD98AC/DOUT -> /PCBMountButtons/sheet5FFD98B2/DIN
- R143 pad 1: /PCBMountButtons/sheet5FFD98B2/DOUT -> /PCBMountButtons/sheet5FFD98C6/DIN
- R144 pad 1: /PCBMountButtons/sheet5FFD98C6/DOUT -> /PCBMountButtons/sheet5FFD98E7/DIN
- R145 pad 1: /PCBMountButtons/sheet5FFD98E7/DOUT -> /PCBMountButtons/sheet5FFD98EE/DIN
- R146 pad 1: /PCBMountButtons/sheet5FFD98EE/DOUT -> /PCBMountButtons/sheet5FFD990E/DIN
- R147 pad 1: /PCBMountButtons/sheet5FFD990E/DOUT -> /PCBMountButtons/sheet5FFD9914/DIN
- R148 pad 1: /PCBMountButtons/sheet5FFD9914/DOUT -> /PCBMountButtons/sheet5FFD9928/DIN
- R149 pad 1: /PCBMountButtons/sheet5FFD9928/DOUT -> /PCBMountButtons/sheet5FFFA930/DIN
- R150 pad 1: /PCBMountButtons/sheet5FFFA930/DOUT -> /PCBMountButtons/sheet5FFFA938/DIN
- R151 pad 1: /PCBMountButtons/sheet5FFFA938/DOUT -> /PCBMountButtons/sheet5FFFA94C/DIN
- R152 pad 1: /PCBMountButtons/sheet5FFFA94C/DOUT -> /PCBMountButtons/sheet5FFFA960/DIN
- R153 pad 1: /PCBMountButtons/sheet5FFFA960/DOUT -> /PCBMountButtons/sheet5FFFA981/DIN
- R154 pad 1: /PCBMountButtons/sheet5FFFA981/DOUT -> /PCBMountButtons/sheet5FFFA987/DIN
- R155 pad 1: /PCBMountButtons/sheet5FFFA987/DOUT -> /PCBMountButtons/sheet5FFFA99B/DIN
- R156 pad 1: /PCBMountButtons/sheet5FFFA99B/DOUT -> /PCBMountButtons/sheet5FFFA9BC/DIN
- R157 pad 1: /PCBMountButtons/sheet5FFFA9BC/DOUT -> /PCBMountButtons/sheet5FFFA9C3/DIN
- R158 pad 1: /PCBMountButtons/sheet5FFFA9C3/DOUT -> /PCBMountButtons/sheet5FFFA9E3/DIN
- R159 pad 1: /PCBMountButtons/sheet5FFFA9E3/DOUT -> /PCBMountButtons/sheet5FFFA9E9/DIN
- R160 pad 1: /PCBMountButtons/sheet5FFFA9E9/DOUT -> /PCBMountButtons/sheet5FFFA9FD/DIN
- R161 pad 1: /PCBMountButtons/sheet5FFFA9FD/DOUT -> /PCBMountButtons/sheet6001C156/DIN
- R162 pad 1: /PCBMountButtons/sheet6001C156/DOUT -> /PCBMountButtons/sheet6001C15E/DIN
- R163 pad 1: /PCBMountButtons/sheet6001C15E/DOUT -> /PCBMountButtons/sheet6001C172/DIN
- R164 pad 1: /PCBMountButtons/sheet6001C172/DOUT -> /PCBMountButtons/sheet6001C186/DIN
- R165 pad 1: /PCBMountButtons/sheet6001C186/DOUT -> /PCBMountButtons/sheet6001C1A7/DIN
- R166 pad 1: /PCBMountButtons/sheet6001C1A7/DOUT -> /PCBMountButtons/sheet6001C1AD/DIN
- R167 pad 1: /PCBMountButtons/sheet6001C1AD/DOUT -> /PCBMountButtons/sheet6001C1C1/DIN
- R168 pad 1: /PCBMountButtons/sheet6001C1C1/DOUT -> /PCBMountButtons/sheet6001C1E2/DIN
- R169 pad 1: /PCBMountButtons/sheet6001C1E2/DOUT -> /PCBMountButtons/sheet6001C1E9/DIN
- R170 pad 1: /PCBMountButtons/sheet6001C1E9/DOUT -> /PCBMountButtons/sheet6112CF44/DIN
- R171 pad 1: /PCBMountButtons/sheet6112CF44/DOUT -> /PCBMountButtons/sheet61155765/DIN
- R172 pad 1: /PCBMountButtons/sheet61155765/DOUT -> /PCBMountButtons/sheet611F5592/DIN
- R173 pad 1: /PCBMountButtons/sheet611F5592/DOUT -> /PCBMountButtons/sheet6120995A/DIN
Routing:
- net BTNX-6: track 0.00 -> 41.7 mm
- net BTNX-3: track 0.00 -> 41.4 mm
- net BTNX-1: track 0.00 -> 40.6 mm
- net BTNX-2: track 0.00 -> 40.4 mm
- net BTN9: track 0.00 -> 38.5 mm
- net BTN7: track 0.00 -> 37.8 mm
- net BTN6: track 0.00 -> 37.7 mm
- net BTN8: track 0.00 -> 37.7 mm
- net BTN5: track 0.00 -> 36.8 mm
- net /PCBMountButtons/sheet6120995A/DIN: track 2.34 -> 23.2 mm
- net /PCBMountButtons/sheet61ACB899/DIN: track 1.27 -> 22.0 mm
- net /PCBMountButtons/sheet6112CF44/DIN: track 2.34 -> 22.8 mm
- net /PCBMountButtons/sheet6001C1E2/DIN: track 2.32 -> 22.7 mm
- net /PCBMountButtons/sheet6001C1C1/DIN: track 2.32 -> 22.7 mm
- net /PCBMountButtons/sheet6001C1AD/DIN: track 2.32 -> 22.6 mm
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
Commit message: routing progress
Parts:
- removed R106, R108, R59, R61, R82, R85, R89: 210R, Resistor_SMD:R_0805_2012Metric
- C1, C10, C11, C13, C14, C15, C17, C18, C19, C2, C23, C29, C30, C31, C32, C33, C34, C35, C36, C37, C38, C39, C40, C41, C42, C43, C44, C45, C46, C47, C48, C49, C5, C50, C55, C56, C57, C58, C59, C60, C61, C62, C63, C64, C7, D1, D10, D11, D12, D13, D14, D15, D16, D17, D18, D2, D3, D4, D5, D6, D7, D9, F1, F2, FB1, FB2, FB3, J17, J20, J21, JP1, JP2, JP3, JP4, JP5, L1, L2, L4, L5, Q2, Q3, R1, R10, R11, R12, R14, R15, R16, R18, R2, R21, R22, R23, R24, R25, R26, R27, R28, R29, R3, R30, R31, R32, R33, R34, R35, R36, R37, R38, R39, R4, R40, R41, R42, R43, R44, R45, R46, R47, R48, R49, R5, R50, R51, R52, R53, R6, R8, R9, TP1, TP10, TP11, TP12, TP13, TP14, TP15, TP16, TP17, TP18, TP19, TP2, TP20, TP21, TP22, TP23, TP24, TP25, TP26, TP3, TP4, TP5, TP6, TP7, TP8, TP9, U1, U3, U4, U5, Y1, Y2, Y3: moved to B.Cu
- R174: moved to F.Cu
- moved TP15 427.7 mm to (-138.5, 92.7)
- moved TP16 427.7 mm to (-141.0, 92.8)
- moved TP21 427.7 mm to (-136.8, 108.1)
- moved TP22 427.7 mm to (-131.9, 105.3)
- moved TP23 427.7 mm to (-131.8, 103.0)
- moved TP24 427.7 mm to (-131.8, 100.3)
- moved TP25 427.7 mm to (-131.7, 97.5)
- moved TP26 427.7 mm to (-139.9, 108.1)
- moved U5 427.7 mm to (-140.3, 99.6)
- moved C43 415.4 mm to (-142.5, 105.3)
- moved R50 411.8 mm to (-146.3, 97.0)
- moved R46 410.6 mm to (-139.4, 90.6)
- moved C46 402.1 mm to (-143.9, 94.7), turned to 180 degrees
- moved R33 401.9 mm to (-149.3, 91.7)
- moved C49 399.1 mm to (-126.9, 101.4)
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- renumbered SW7 to SW10, SW6 to SW11, SW26 to SW19, SW25 to SW20, SW24 to SW21, SW23 to SW22, SW22 to SW23, SW21 to SW24, SW20 to SW25, SW19 to SW26, SW43 to SW36, SW42 to SW37, SW41 to SW38, SW40 to SW39, SW39 to SW40, SW38 to SW41, SW37 to SW42, SW36 to SW43, SW56 to SW51, SW55 to SW52, SW54 to SW53, SW53 to SW54, SW52 to SW55, SW51 to SW56, SW11 to SW6, SW10 to SW7, SW9 to SW8, SW8 to SW9
Connections:
- SW10 pad 1: BTN11 -> BTN14
- SW11 pad 1: BTN10 -> BTN15
- SW19 pad 1: BTN30 -> BTN23
- SW20 pad 1: BTN29 -> BTN24
- SW21 pad 1: BTN28 -> BTN25
- SW22 pad 1: BTN27 -> BTN26
- SW23 pad 1: BTN26 -> BTN27
- SW24 pad 1: BTN25 -> BTN28
- SW25 pad 1: BTN24 -> BTN29
- SW26 pad 1: BTN23 -> BTN30
- SW36 pad 1: BTN47 -> BTN40
- SW37 pad 1: BTN46 -> BTN41
- SW38 pad 1: BTN45 -> BTN42
- SW39 pad 1: BTN44 -> BTN43
- SW40 pad 1: BTN43 -> BTN44
- SW41 pad 1: BTN42 -> BTN45
- SW42 pad 1: BTN41 -> BTN46
- SW43 pad 1: BTN40 -> BTN47
- SW51 pad 1: BTN60 -> BTN55
- SW52 pad 1: BTN59 -> BTN56
- SW53 pad 1: BTN58 -> BTN57
- SW54 pad 1: BTN57 -> BTN58
- SW55 pad 1: BTN56 -> BTN59
- SW56 pad 1: BTN55 -> BTN60
- SW6 pad 1: BTN15 -> BTN10
- SW7 pad 1: BTN14 -> BTN11
- SW8 pad 1: BTN13 -> BTN12
- SW9 pad 1: BTN12 -> BTN13
- U4 pad : (no net) -> GND
Routing:
- net BTN15: track 13.1 -> 157.3 mm, vias 0 -> 3
- net BTN11: track 0.00 -> 143.8 mm, vias 0 -> 1
- net BTNX-1: track 40.6 -> 176.6 mm, vias 0 -> 3
- net BTN5: track 36.8 -> 166.6 mm, vias 0 -> 1
- net BTN17: track 0.00 -> 128.6 mm, vias 0 -> 1
- net BTN9: track 38.5 -> 166.4 mm, vias 0 -> 3
- net BTNX-6: track 41.7 -> 167.6 mm, vias 0 -> 1
- net BTN18: track 0.00 -> 119.3 mm, vias 0 -> 3
- net BTN14: track 13.2 -> 129.6 mm, vias 0 -> 3
- net BTN13: track 12.9 -> 129.1 mm, vias 0 -> 1
- net BTNX-2: track 40.4 -> 154.2 mm, vias 0 -> 1
- net BTN8: track 37.7 -> 151.4 mm, vias 0 -> 3
- net BTN6: track 37.7 -> 148.2 mm, vias 0 -> 1
- net BTN12: track 0.00 -> 108.2 mm, vias 0 -> 1
- net BTN54: track 0.00 -> 103.2 mm
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- added copper zone on In1.Cu, net GND
- added copper zone on In2.Cu, net VLED
Other:
- copper layers 2 -> 4

Commit message: Moves meta button connectors to correct spots
Updates locations for layout to continue
Parts:
- removed C1, C2: DNP-1uF 25V, Capacitor_SMD:C_0805_2012Metric
- removed C11: 1uF 25V, Capacitor_SMD:C_0805_2012Metric
- removed D3: 5Vw, Package_TO_SOT_SMD:SOT-23
- removed J2: SDS-50J, rainboard_fp:CUI_SDS-50J
- removed R1, R8: 210R, Resistor_SMD:R_0805_2012Metric
- removed R4: 11R, Resistor_SMD:R_0603_1608Metric
- removed U1: 6N137, rainboard_fp:COUPL_6N138SDM
- C51, C52, C53, C54: moved to B.Cu
- J1, J15, J3: moved to F.Cu
- moved C41 55.9 mm to (177.1, 97.7)
- moved R37 55.9 mm to (141.6, 131.6)
- moved R38 55.9 mm to (141.1, 145.3)
- moved C29 55.9 mm to (148.3, 139.8)
- moved D14 55.9 mm to (151.6, 133.9)
- moved D15 55.9 mm to (150.9, 127.5)
- moved L5 55.9 mm to (172.3, 98.4)
- moved R36 55.9 mm to (140.9, 141.1)
- moved C39 55.9 mm to (168.0, 97.9)
- moved C40 55.9 mm to (168.4, 101.1)
- moved C42 55.9 mm to (169.7, 107.9)
- moved R35 55.9 mm to (141.0, 136.9)
- moved J12 44.6 mm to (-101.0, 8.58), turned to 120 degrees
- moved J16 42.5 mm to (-56.8, 85.4), turned to 120 degrees
- moved J14 38.6 mm to (-71.6, 59.8), turned to 120 degrees
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Connections:
- U3 pad 5: Net-(R8-Pad1) -> GND
- U3 pad 8: MIDI-IN -> Net-(U3-Pad8)
- U3 pad 9: Net-(U3-Pad6) -> GND
- U4 pad : GND -> (no net)
- U6 pad 45: MIDI-IN -> Net-(U6-Pad45)
